File: robot/motorboard/v1.0.0/motorboard/_autosave-drive_motor_digital.kicad_sch (KiCad schematic)
At the start: 11 parts

Commit message: motor bridge cleanup
Connections:
- net HALL_A: now also J?.2 (Pin_2), R?.2
- net HALL_B: now also J?.3 (Pin_3), R?.2
- net HALL_C: now also J?.4 (Pin_4), R?.2
- net at J?.2 (Pin_2): no longer U?.17 (PA6/GPIO/T3C1/ADC6)
- net at J?.3 (Pin_3): no longer U?.18 (PA7/GPIO/T3C2/ADC7)
- net ENC_I: now reaches U?.19 (PB1/GPIO/T3C4/ADC9)
- net SWDIO: now reaches U?.37 (PA13/SWDIO)
- net UART_TX renamed SWDCLK
- new net ENC_A: U?.17 (PA6/GPIO/T3C1/ADC6)
- new net ENC_B: U?.18 (PA7/GPIO/T3C2/ADC7)
Changed lines of the file:
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@@
   (junction (at 121.92 57.15) (diameter 0.9144) (color 0 0 0 0))
   (junction (at 121.92 105.41) (diameter 0.9144) (color 0 0 0 0))
+  (junction (at 185.42 102.87) (diameter 0.9144) (color 0 0 0 0))
   (junction (at 261.62 49.53) (diameter 0.9144) (color 0 0 0 0))
+  (junction (at 261.62 62.23) (diameter 0.9144) (color 0 0 0 0))
   (junction (at 273.05 49.53) (diameter 0.9144) (color 0 0 0 0))
+  (junction (at 273.05 64.77) (diameter 0.9144) (color 0 0 0 0))
   (junction (at 284.48 49.53) (diameter 0.9144) (color 0 0 0 0))
+  (junction (at 284.48 67.31) (diameter 0.9144) (color 0 0 0 0))
   (bus_entry (at 189.23 64.77) (size 2.54 2.54)
     (stroke (width 0) (type solid) (color 0 0 0 0))
@@
     (stroke (width 0) (type solid) (color 0 0 0 0))
   )
+  (bus_entry (at 189.23 80.01) (size 2.54 2.54)
+    (stroke (width 0) (type solid) (color 0 0 0 0))
+  )
+  (bus_entry (at 189.23 82.55) (size 2.54 2.54)
+    (stroke (width 0) (type solid) (color 0 0 0 0))
+  )
+  (bus_entry (at 189.23 85.09) (size 2.54 2.54)
+    (stroke (width 0) (type solid) (color 0 0 0 0))
+  )
   (wire (pts (xy 27.94 57.15) (xy 40.64 57.15))
     (stroke (width 0) (type solid) (color 0 0 0 0))
@@
     (stroke (width 0) (type solid) (color 0 0 0 0))
   )
-  (wire (pts (xy 180.34 80.01) (xy 186.69 80.01))
-    (stroke (width 0) (type solid) (color 0 0 0 0))
-  )
-  (wire (pts (xy 180.34 102.87) (xy 187.96 102.87))
+  (wire (pts (xy 180.34 80.01) (xy 189.23 80.01))
+    (stroke (width 0) (type solid) (color 0 0 0 0))
+  )
+  (wire (pts (xy 180.34 82.55) (xy 189.23 82.55))
+    (stroke (width 0) (type solid) (color 0 0 0 0))
+  )
+  (wire (pts (xy 180.34 85.09) (xy 189.23 85.09))
+    (stroke (width 0) (type solid) (color 0 0 0 0))
+  )
+  (wire (pts (xy 180.34 102.87) (xy 185.42 102.87))
     (stroke (width 0) (type solid) (color 0 0 0 0))
   )
@@
     (stroke (width 0) (type solid) (color 0 0 0 0))
   )
-  (wire (pts (xy 184.15 82.55) (xy 180.34 82.55))
-    (stroke (width 0) (type solid) (color 0 0 0 0))
-  )
-  (wire (pts (xy 184.15 87.63) (xy 184.15 82.55))
-    (stroke (width 0) (type solid) (color 0 0 0 0))
-  )
-  (wire (pts (xy 186.69 80.01) (xy 186.69 85.09))
-    (stroke (width 0) (type solid) (color 0 0 0 0))
-  )
-  (wire (pts (xy 186.69 85.09) (xy 231.14 85.09))
-    (stroke (width 0) (type solid) (color 0 0 0 0))
-  )
-  (wire (pts (xy 228.6 87.63) (xy 184.15 87.63))
-    (stroke (width 0) (type solid) (color 0 0 0 0))
-  )
-  (wire (pts (xy 228.6 96.52) (xy 228.6 87.63))
-    (stroke (width 0) (type solid) (color 0 0 0 0))
-  )
-  (wire (pts (xy 228.6 96.52) (xy 256.54 96.52))
-    (stroke (width 0) (type solid) (color 0 0 0 0))
-  )
-  (wire (pts (xy 231.14 85.09) (xy 231.14 93.98))
-    (stroke (width 0) (type solid) (color 0 0 0 0))
-  )
-  (wire (pts (xy 231.14 93.98) (xy 256.54 93.98))
+  (wire (pts (xy 182.88 97.79) (xy 182.88 100.33))
+    (stroke (width 0) (type solid) (color 0 0 0 0))
+  )
+  (wire (pts (xy 182.88 100.33) (xy 180.34 100.33))
+    (stroke (width 0) (type solid) (color 0 0 0 0))
+  )
+  (wire (pts (xy 185.42 100.33) (xy 185.42 102.87))
+    (stroke (width 0) (type solid) (color 0 0 0 0))
+  )
+  (wire (pts (xy 185.42 102.87) (xy 187.96 102.87))
+    (stroke (width 0) (type solid) (color 0 0 0 0))
+  )
+  (wire (pts (xy 187.96 97.79) (xy 182.88 97.79))
+    (stroke (width 0) (type solid) (color 0 0 0 0))
+  )
+  (wire (pts (xy 187.96 100.33) (xy 185.42 100.33))
     (stroke (width 0) (type solid) (color 0 0 0 0))
   )
@@
     (stroke (width 0) (type solid) (color 0 0 0 0))
   )
+  (wire (pts (xy 257.81 62.23) (xy 261.62 62.23))
+    (stroke (width 0) (type solid) (color 0 0 0 0))
+  )
+  (wire (pts (xy 257.81 64.77) (xy 273.05 64.77))
+    (stroke (width 0) (type solid) (color 0 0 0 0))
+  )
+  (wire (pts (xy 257.81 67.31) (xy 284.48 67.31))
+    (stroke (width 0) (type solid) (color 0 0 0 0))
+  )
   (wire (pts (xy 261.62 49.53) (xy 261.62 52.07))
     (stroke (width 0) (type solid) (color 0 0 0 0))
@@
   )
   (bus (pts (xy 191.77 81.28) (xy 195.58 81.28))
+    (stroke (width 0) (type solid) (color 0 0 0 0))
+  )
+  (bus (pts (xy 191.77 82.55) (xy 191.77 88.9))
+    (stroke (width 0) (type solid) (color 0 0 0 0))
+  )
+  (bus (pts (xy 191.77 88.9) (xy 195.58 88.9))
     (stroke (width 0) (type solid) (color 0 0 0 0))
   )
@@
     (effects (font (size 1.27 1.27)) (justify right bottom))
   )
+  (label "ENC_A" (at 189.23 80.01 180)
+    (effects (font (size 1.27 1.27)) (justify right bottom))
+  )
+  (label "ENC_B" (at 189.23 82.55 180)
+    (effects (font (size 1.27 1.27)) (justify right bottom))
+  )
+  (label "ENC_I" (at 189.23 85.09 180)
+    (effects (font (size 1.27 1.27)) (justify right bottom))
+  )
   (label "HALL" (at 195.58 73.66 0)
     (effects (font (size 1.27 1.27)) (justify left bottom))
   )
+  (label "ENC" (at 195.58 88.9 0)
+    (effects (font (size 1.27 1.27)) (justify left bottom))
+  )
+  (label "HALL_A" (at 257.81 62.23 180)
+    (effects (font (size 1.27 1.27)) (justify right bottom))
+  )
+  (label "HALL_B" (at 257.81 64.77 180)
+    (effects (font (size 1.27 1.27)) (justify right bottom))
+  )
+  (label "HALL_C" (at 257.81 67.31 180)
+    (effects (font (size 1.27 1.27)) (justify right bottom))
+  )
   (hierarchical_label "VDD" (shape input) (at 27.94 57.15 180)
     (effects (font (size 1.27 1.27)) (justify right))
@@
     (effects (font (size 1.27 1.27)) (justify right))
   )
+  (hierarchical_label "SWDIO" (shape bidirectional) (at 187.96 97.79 0)
+    (effects (font (size 1.27 1.27)) (justify left))
+  )
+  (hierarchical_label "SWDCLK" (shape input) (at 187.96 100.33 0)
+    (effects (font (size 1.27 1.27)) (justify left))
+  )
   (hierarchical_label "UART_TX" (shape output) (at 187.96 102.87 0)
