File: robot/motorboard/v1.0.0/motorboard/drive_motor_digital.kicad_sch (KiCad schematic)
At the start: 13 parts, among them J14 Conn_01x05_Female, J15 Conn_01x06_Female, U6 STSPIN32F0A

Commit message: more footprint assignments
Parts:
- D6: footprint (none) -> LED_SMD:LED_0603_1608Metric_Pad1.05x0.95mm_HandSolder
- R41, R42, R43, R44, R45: footprint (none) -> Resistor_SMD:R_0402_1005Metric_Pad0.72x0.64mm_HandSolder
Changed lines of the file:
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@@
   (symbol (lib_id "power:PWR_FLAG") (at 62.23 31.75 0)
     (in_bom yes) (on_board yes) (fields_autoplaced)
-    (property "Reference" "#FLG03" (id 0) (at 62.23 29.845 0)
+    (property "Reference" "#FLG012" (id 0) (at 62.23 29.845 0)
       (effects (font (size 1.27 1.27)) hide)
     )
@@
   (symbol (lib_id "power:PWR_FLAG") (at 62.23 63.5 0)
     (in_bom yes) (on_board yes) (fields_autoplaced)
-    (property "Reference" "#FLG04" (id 0) (at 62.23 61.595 0)
+    (property "Reference" "#FLG013" (id 0) (at 62.23 61.595 0)
       (effects (font (size 1.27 1.27)) hide)
     )
@@
   (symbol (lib_id "power:GND") (at 62.23 49.53 0)
     (in_bom yes) (on_board yes)
-    (property "Reference" "#PWR063" (id 0) (at 62.23 55.88 0)
+    (property "Reference" "#PWR0123" (id 0) (at 62.23 55.88 0)
       (effects (font (size 1.27 1.27)) hide)
     )
@@
   (symbol (lib_id "power:GND") (at 62.23 78.74 0)
     (in_bom yes) (on_board yes) (fields_autoplaced)
-    (property "Reference" "#PWR064" (id 0) (at 62.23 85.09 0)
+    (property "Reference" "#PWR0124" (id 0) (at 62.23 85.09 0)
       (effects (font (size 1.27 1.27)) hide)
     )
@@
   (symbol (lib_id "power:GND") (at 73.66 154.94 0)
     (in_bom yes) (on_board yes)
-    (property "Reference" "#PWR065" (id 0) (at 73.66 161.29 0)
+    (property "Reference" "#PWR0125" (id 0) (at 73.66 161.29 0)
       (effects (font (size 1.27 1.27)) hide)
     )
@@
   (symbol (lib_id "power:GND") (at 111.76 93.98 0)
     (in_bom yes) (on_board yes) (fields_autoplaced)
-    (property "Reference" "#PWR067" (id 0) (at 111.76 100.33 0)
+    (property "Reference" "#PWR0127" (id 0) (at 111.76 100.33 0)
       (effects (font (size 1.27 1.27)) hide)
     )
@@
   (symbol (lib_id "power:GND") (at 172.72 147.32 0)
     (in_bom yes) (on_board yes) (fields_autoplaced)
-    (property "Reference" "#PWR066" (id 0) (at 172.72 153.67 0)
+    (property "Reference" "#PWR0126" (id 0) (at 172.72 153.67 0)
       (effects (font (size 1.27 1.27)) hide)
     )
@@
   (symbol (lib_id "power:GND") (at 252.73 142.24 0)
     (in_bom yes) (on_board yes) (fields_autoplaced)
-    (property "Reference" "#PWR068" (id 0) (at 252.73 148.59 0)
+    (property "Reference" "#PWR0128" (id 0) (at 252.73 148.59 0)
       (effects (font (size 1.27 1.27)) hide)
     )
@@
       (effects (font (size 1.27 1.27)) (justify left))
     )
-    (property "Footprint" "" (id 2) (at 37.846 138.684 90)
+    (property "Footprint" "Resistor_SMD:R_0402_1005Metric_Pad0.72x0.64mm_HandSolder" (id 2) (at 37.846 138.684 90)
       (effects (font (size 1.27 1.27)) hide)
     )
@@
       (effects (font (size 1.27 1.27)) (justify left))
     )
-    (property "Footprint" "" (id 2) (at 49.276 138.684 90)
+    (property "Footprint" "Resistor_SMD:R_0402_1005Metric_Pad0.72x0.64mm_HandSolder" (id 2) (at 49.276 138.684 90)
       (effects (font (size 1.27 1.27)) hide)
     )
@@
       (effects (font (size 1.27 1.27)) (justify left))
     )
-    (property "Footprint" "" (id 2) (at 60.706 138.684 90)
+    (property "Footprint" "Resistor_SMD:R_0402_1005Metric_Pad0.72x0.64mm_HandSolder" (id 2) (at 60.706 138.684 90)
       (effects (font (size 1.27 1.27)) hide)
     )
@@
       (effects (font (size 1.27 1.27)) (justify left))
     )
-    (property "Footprint" "" (id 2) (at 108.966 39.624 90)
+    (property "Footprint" "Resistor_SMD:R_0402_1005Metric_Pad0.72x0.64mm_HandSolder" (id 2) (at 108.966 39.624 90)
       (effects (font (size 1.27 1.27)) hide)
     )
@@
     (property "Reference" "R45" (id 0) (at 232.41 132.08 90))
     (property "Value" "1k" (id 1) (at 232.41 134.62 90))
-    (property "Footprint" "" (id 2) (at 232.664 137.414 90)
+    (property "Footprint" "Resistor_SMD:R_0402_1005Metric_Pad0.72x0.64mm_HandSolder" (id 2) (at 232.664 137.414 90)
       (effects (font (size 1.27 1.27)) hide)
     )
@@
     (property "Reference" "D6" (id 0) (at 245.3005 130.81 0))
     (property "Value" "RED" (id 1) (at 245.3005 133.35 0))
-    (property "Footprint" "" (id 2) (at 245.11 138.43 0)
-      (effects (font (size 1.27 1.27)) hide)
-    )
+    (property "Footprint" "LED_SMD:LED_0603_1608Metric_Pad1.05x0.95mm_HandSolder" (id 2) (at 245.11 138.43 0)
+      (effects (font (size 1.27 1.27)) hide)
+    )

Commit message: updated file formates to v6.0.0-rc2
Parts:
- renumbered C15 to C49, C16 to C50, C17 to C51, C18 to C52, D6 to D20, J14 to J20, J15 to J21, R41 to R119, R42 to R120, R43 to R121, R44 to R122, R45 to R123, U6 to U8

Commit message: reannotation
Parts:
- renumbered C49 to C34, C50 to C35, C51 to C36, C52 to C37, D20 to D13, J20 to J17, J21 to J18, R119 to R83, R120 to R84, R121 to R85, R122 to R86, R123 to R87
Changed lines of the file:
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@@
   (symbol (lib_id "Device:C") (at 62.23 72.39 0)
     (in_bom yes) (on_board yes) (fields_autoplaced)
-    (property "Reference" "C51" (id 0) (at 66.04 71.1199 0)
+    (property "Reference" "C36" (id 0) (at 66.04 71.1199 0)
       (effects (font (size 1.27 1.27)) (justify left))
     )
@@
   (symbol (lib_id "Device:R_US") (at 232.41 138.43 90)
     (in_bom yes) (on_board yes) (fields_autoplaced)
-    (property "Reference" "R123" (id 0) (at 232.41 132.08 90))
+    (property "Reference" "R87" (id 0) (at 232.41 132.08 90))
     (property "Value" "1k" (id 1) (at 232.41 134.62 90))
     (property "Footprint" "Resistor_SMD:R_0402_1005Metric_Pad0.72x0.64mm_HandSolder" (id 2) (at 232.664 137.414 90)
@@
   (symbol (lib_id "power:GND") (at 111.76 93.98 0)
     (in_bom yes) (on_board yes) (fields_autoplaced)
-    (property "Reference" "#PWR0107" (id 0) (at 111.76 100.33 0)
+    (property "Reference" "#PWR093" (id 0) (at 111.76 100.33 0)
       (effects (font (size 1.27 1.27)) hide)
     )
@@
   (symbol (lib_id "Device:LED") (at 245.11 138.43 180)
     (in_bom yes) (on_board yes) (fields_autoplaced)
-    (property "Reference" "D20" (id 0) (at 245.3005 130.81 0))
+    (property "Reference" "D13" (id 0) (at 245.3005 130.81 0))
     (property "Value" "RED" (id 1) (at 245.3005 133.35 0))
     (property "Footprint" "LED_SMD:LED_0603_1608Metric_Pad1.05x0.95mm_HandSolder" (id 2) (at 245.11 138.43 0)
@@
   (symbol (lib_id "Device:R_US") (at 36.83 138.43 0)
     (in_bom yes) (on_board yes) (fields_autoplaced)
-    (property "Reference" "R119" (id 0) (at 39.37 137.1599 0)
+    (property "Reference" "R83" (id 0) (at 39.37 137.1599 0)
       (effects (font (size 1.27 1.27)) (justify left))
     )
@@
   (symbol (lib_id "power:GND") (at 172.72 147.32 0)
     (in_bom yes) (on_board yes) (fields_autoplaced)
-    (property "Reference" "#PWR0106" (id 0) (at 172.72 153.67 0)
+    (property "Reference" "#PWR094" (id 0) (at 172.72 153.67 0)
       (effects (font (size 1.27 1.27)) hide)
     )
@@
   (symbol (lib_id "Device:C") (at 111.76 69.85 0)
     (in_bom yes) (on_board yes) (fields_autoplaced)
-    (property "Reference" "C52" (id 0) (at 115.57 68.5799 0)
+    (property "Reference" "C37" (id 0) (at 115.57 68.5799 0)
       (effects (font (size 1.27 1.27)) (justify left))
     )
@@
   (symbol (lib_id "power:GND") (at 73.66 154.94 0)
     (in_bom yes) (on_board yes)
-    (property "Reference" "#PWR0105" (id 0) (at 73.66 161.29 0)
+    (property "Reference" "#PWR092" (id 0) (at 73.66 161.29 0)
       (effects (font (size 1.27 1.27)) hide)
     )
@@
   (symbol (lib_id "power:PWR_FLAG") (at 62.23 63.5 0)
     (in_bom yes) (on_board yes) (fields_autoplaced)
-    (property "Reference" "#FLG010" (id 0) (at 62.23 61.595 0)
+    (property "Reference" "#FLG08" (id 0) (at 62.23 61.595 0)
       (effects (font (size 1.27 1.27)) hide)
     )
@@
   (symbol (lib_id "Device:C") (at 62.23 40.64 0)
     (in_bom yes) (on_board yes) (fields_autoplaced)
-    (property "Reference" "C50" (id 0) (at 66.04 39.3699 0)
+    (property "Reference" "C35" (id 0) (at 66.04 39.3699 0)
       (effects (font (size 1.27 1.27)) (justify left))
     )
@@
   (symbol (lib_id "Connector:Conn_01x06_Female") (at 179.07 137.16 0)
     (in_bom yes) (on_board yes) (fields_autoplaced)
-    (property "Reference" "J21" (id 0) (at 180.34 137.1599 0)
+    (property "Reference" "J18" (id 0) (at 180.34 137.1599 0)
       (effects (font (size 1.27 1.27)) (justify left))
     )
@@
   (symbol (lib_id "power:GND") (at 252.73 142.24 0)
     (in_bom yes) (on_board yes) (fields_autoplaced)
-    (property "Reference" "#PWR0108" (id 0) (at 252.73 148.59 0)
+    (property "Reference" "#PWR095" (id 0) (at 252.73 148.59 0)
       (effects (font (size 1.27 1.27)) hide)
     )
@@
   (symbol (lib_id "Connector:Conn_01x05_Female") (at 80.01 147.32 0)
     (in_bom yes) (on_board yes) (fields_autoplaced)
-    (property "Reference" "J20" (id 0) (at 81.28 146.0499 0)
+    (property "Reference" "J17" (id 0) (at 81.28 146.0499 0)
       (effects (font (size 1.27 1.27)) (justify left))
     )
@@
   (symbol (lib_id "Device:R_US") (at 59.69 138.43 0)
     (in_bom yes) (on_board yes) (fields_autoplaced)
-    (property "Reference" "R121" (id 0) (at 62.23 137.1599 0)
+    (property "Reference" "R85" (id 0) (at 62.23 137.1599 0)
       (effects (font (size 1.27 1.27)) (justify left))
     )
@@
   (symbol (lib_id "Device:R_US") (at 48.26 138.43 0)
     (in_bom yes) (on_board yes) (fields_autoplaced)
-    (property "Reference" "R120" (id 0) (at 50.8 137.1599 0)
+    (property "Reference" "R84" (id 0) (at 50.8 137.1599 0)
       (effects (font (size 1.27 1.27)) (justify left))
     )
@@
   (symbol (lib_id "Device:C") (at 44.45 40.64 0)
     (in_bom yes) (on_board yes) (fields_autoplaced)
-    (property "Reference" "C49" (id 0) (at 48.26 39.3699 0)
+    (property "Reference" "C34" (id 0) (at 48.26 39.3699 0)
       (effects (font (size 1.27 1.27)) (justify left))
     )
@@
   (symbol (lib_id "power:GND") (at 62.23 78.74 0)
     (in_bom yes) (on_board yes) (fields_autoplaced)
-    (property "Reference" "#PWR0104" (id 0) (at 62.23 85.09 0)
+    (property "Reference" "#PWR091" (id 0) (at 62.23 85.09 0)
       (effects (font (size 1.27 1.27)) hide)
     )
@@
   (symbol (lib_id "Device:R_US") (at 107.95 39.37 0)
     (in_bom yes) (on_board yes) (fields_autoplaced)
-    (property "Reference" "R122" (id 0) (at 110.49 38.0999 0)
+    (property "Reference" "R86" (id 0) (at 110.49 38.0999 0)
       (effects (font (size 1.27 1.27)) (justify left))
     )
@@
   (symbol (lib_id "power:GND") (at 62.23 49.53 0)
     (in_bom yes) (on_board yes)
-    (property "Reference" "#PWR0103" (id 0) (at 62.23 55.88 0)
+    (property "Reference" "#PWR090" (id 0) (at 62.23 55.88 0)
       (effects (font (size 1.27 1.27)) hide)
     )
@@
   (symbol (lib_id "power:PWR_FLAG") (at 62.23 31.75 0)
     (in_bom yes) (on_board yes) (fields_autoplaced)
-    (property "Reference" "#FLG09" (id 0) (at 62.23 29.845 0)
-      (effects (font (size 1.27 1.27)) hide)
-    )
+    (property "Reference" "#FLG07" (id 0) (at 62.23 29.845 0)
+      (effects (font (size 1.27 1.27)) hide)
+    )
