File: robot/kicker/v1.0.0/kicker/kicker.kicad_pcb (KiCad board)
At the start: 4 copper layers, 76 x 90 mm, 136 parts, among them J1 XT30PW-M, J2 1054052108, J3 2157601002, J4 2157601002, J5 Conn_ARM_JTAG_SWD_10, J6 Conn_01x03, J7 Conn_01x03, Q1 BSC0402NSATMA1, Q2 IXGA48N60A3, Q3 IXGA48N60A3, Q4 BSS138K, SW1 TS02-66-73-BK-160-SCR-D, U1 LM1117-5.0, U2 LM1117-3.3, U3 ADUM7441, U4 LT3751-QFN, U5 IX4427, U6 STM32F030K6Tx, U7 SK9822, U8 SK9822

Commit message: routing work
Routing:
- net GND: vias 111 -> 140
Changed lines of the file:
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@@
   (via (at 240.8 140.2) (size 0.8) (drill 0.3) (layers "F.Cu" "B.Cu") (free) (net 2))
   (via (at 226.475 168.725) (size 0.8) (drill 0.3) (layers "F.Cu" "B.Cu") (free) (net 2))
+  (via (at 217.8 119.2) (size 0.8) (drill 0.3) (layers "F.Cu" "B.Cu") (free) (net 2))
+  (via (at 216.8 120.2) (size 0.8) (drill 0.3) (layers "F.Cu" "B.Cu") (free) (net 2))
   (via (at 231.4 162.4) (size 0.8) (drill 0.3) (layers "F.Cu" "B.Cu") (net 2))
   (via (at 238.8 138.2) (size 0.8) (drill 0.3) (layers "F.Cu" "B.Cu") (free) (net 2))
   (via (at 240.8 166.2) (size 0.8) (drill 0.3) (layers "F.Cu" "B.Cu") (free) (net 2))
+  (via (at 200.8 122.8) (size 0.8) (drill 0.3) (layers "F.Cu" "B.Cu") (free) (net 2))
   (via (at 239.8 152.2) (size 0.8) (drill 0.3) (layers "F.Cu" "B.Cu") (free) (net 2))
   (via (at 219.8 193.2) (size 0.8) (drill 0.3) (layers "F.Cu" "B.Cu") (net 2))
@@
   (via (at 225.55 135.2625) (size 0.8) (drill 0.3) (layers "F.Cu" "B.Cu") (free) (net 2))
   (via (at 216.275 167.725) (size 0.8) (drill 0.3) (layers "F.Cu" "B.Cu") (free) (net 2))
+  (via (at 200.8 120.2) (size 0.8) (drill 0.3) (layers "F.Cu" "B.Cu") (free) (net 2))
   (via (at 240.8 155.2) (size 0.8) (drill 0.3) (layers "F.Cu" "B.Cu") (free) (net 2))
+  (via (at 199.8 120.2) (size 0.8) (drill 0.3) (layers "F.Cu" "B.Cu") (free) (net 2))
   (via (at 238.8 152.2) (size 0.8) (drill 0.3) (layers "F.Cu" "B.Cu") (free) (net 2))
   (via (at 217.675 165.925) (size 0.8) (drill 0.3) (layers "F.Cu" "B.Cu") (free) (net 2))
@@
   (via (at 240.8 141.2) (size 0.8) (drill 0.3) (layers "F.Cu" "B.Cu") (free) (net 2))
   (via (at 238.8 143.2) (size 0.8) (drill 0.3) (layers "F.Cu" "B.Cu") (free) (net 2))
+  (via (at 218.8 122.8) (size 0.8) (drill 0.3) (layers "F.Cu" "B.Cu") (free) (net 2))
   (via (at 240.8 153.2) (size 0.8) (drill 0.3) (layers "F.Cu" "B.Cu") (free) (net 2))
+  (via (at 215.8 122.8) (size 0.8) (drill 0.3) (layers "F.Cu" "B.Cu") (free) (net 2))
   (via (at 226.475 167.725) (size 0.8) (drill 0.3) (layers "F.Cu" "B.Cu") (free) (net 2))
   (via (at 223.475 170.725) (size 0.8) (drill 0.3) (layers "F.Cu" "B.Cu") (free) (net 2))
@@
   (via (at 224.55 136.2625) (size 0.8) (drill 0.3) (layers "F.Cu" "B.Cu") (free) (net 2))
   (via (at 239.8 139.2) (size 0.8) (drill 0.3) (layers "F.Cu" "B.Cu") (free) (net 2))
+  (via (at 216.8 119.2) (size 0.8) (drill 0.3) (layers "F.Cu" "B.Cu") (free) (net 2))
+  (via (at 218.8 120.2) (size 0.8) (drill 0.3) (layers "F.Cu" "B.Cu") (free) (net 2))
   (via (at 220.15 164.2625) (size 0.8) (drill 0.3) (layers "F.Cu" "B.Cu") (net 2))
   (via (at 239.8 154.2) (size 0.8) (drill 0.3) (layers "F.Cu" "B.Cu") (free) (net 2))
@@
   (via (at 238.8 139.2) (size 0.8) (drill 0.3) (layers "F.Cu" "B.Cu") (free) (net 2))
   (via (at 238.8 166.2) (size 0.8) (drill 0.3) (layers "F.Cu" "B.Cu") (free) (net 2))
+  (via (at 198.8 120.2) (size 0.8) (drill 0.3) (layers "F.Cu" "B.Cu") (free) (net 2))
   (via (at 240.8 152.2) (size 0.8) (drill 0.3) (layers "F.Cu" "B.Cu") (free) (net 2))
   (via (at 238.8 169.2) (size 0.8) (drill 0.3) (layers "F.Cu" "B.Cu") (free) (net 2))
@@
   (via (at 239.8 141.2) (size 0.8) (drill 0.3) (layers "F.Cu" "B.Cu") (free) (net 2))
   (via (at 239.8 142.2) (size 0.8) (drill 0.3) (layers "F.Cu" "B.Cu") (free) (net 2))
+  (via (at 219.8 119.2) (size 0.8) (drill 0.3) (layers "F.Cu" "B.Cu") (free) (net 2))
   (via (at 240.8 138.2) (size 0.8) (drill 0.3) (layers "F.Cu" "B.Cu") (free) (net 2))
+  (via (at 215.8 119.2) (size 0.8) (drill 0.3) (layers "F.Cu" "B.Cu") (free) (net 2))
   (via (at 225.475 167.725) (size 0.8) (drill 0.3) (layers "F.Cu" "B.Cu") (free) (net 2))
   (via (at 224.6 182.6) (size 0.8) (drill 0.3) (layers "F.Cu" "B.Cu") (net 2))
   (via (at 223.475 171.725) (size 0.8) (drill 0.3) (layers "F.Cu" "B.Cu") (free) (net 2))
+  (via (at 197.8 122.8) (size 0.8) (drill 0.3) (layers "F.Cu" "B.Cu") (free) (net 2))
   (via (at 233 171.2) (size 0.8) (drill 0.3) (layers "F.Cu" "B.Cu") (net 2))
   (via (at 238.8 140.2) (size 0.8) (drill 0.3) (layers "F.Cu" "B.Cu") (free) (net 2))
@@
   (via (at 240.8 156.2) (size 0.8) (drill 0.3) (layers "F.Cu" "B.Cu") (free) (net 2))
   (via (at 240.8 170.2) (size 0.8) (drill 0.3) (layers "F.Cu" "B.Cu") (free) (net 2))
+  (via (at 217.8 120.2) (size 0.8) (drill 0.3) (layers "F.Cu" "B.Cu") (free) (net 2))
   (via (at 238.8 170.2) (size 0.8) (drill 0.3) (layers "F.Cu" "B.Cu") (free) (net 2))
   (via (at 225.475 170.725) (size 0.8) (drill 0.3) (layers "F.Cu" "B.Cu") (free) (net 2))
+  (via (at 201.8 120.2) (size 0.8) (drill 0.3) (layers "F.Cu" "B.Cu") (free) (net 2))
   (via (at 229.55 137.2625) (size 0.8) (drill 0.3) (layers "F.Cu" "B.Cu") (free) (net 2))
   (via (at 227.475 169.725) (size 0.8) (drill 0.3) (layers "F.Cu" "B.Cu") (free) (net 2))
   (via (at 239.8 143.2) (size 0.8) (drill 0.3) (layers "F.Cu" "B.Cu") (free) (net 2))
+  (via (at 199.8 119.2) (size 0.8) (drill 0.3) (layers "F.Cu" "B.Cu") (free) (net 2))
   (via (at 239.8 153.2) (size 0.8) (drill 0.3) (layers "F.Cu" "B.Cu") (free) (net 2))
   (via (at 238.8 168.2) (size 0.8) (drill 0.3) (layers "F.Cu" "B.Cu") (free) (net 2))
@@
   (via (at 225.475 169.725) (size 0.8) (drill 0.3) (layers "F.Cu" "B.Cu") (free) (net 2))
   (via (at 238.8 142.2) (size 0.8) (drill 0.3) (layers "F.Cu" "B.Cu") (free) (net 2))
-  (via (at 198 120) (size 0.8) (drill 0.3) (layers "F.Cu" "B.Cu") (free) (net 2))
+  (via (at 219.8 122.8) (size 0.8) (drill 0.3) (layers "F.Cu" "B.Cu") (free) (net 2))
   (via (at 227.475 168.725) (size 0.8) (drill 0.3) (layers "F.Cu" "B.Cu") (free) (net 2))
   (via (at 223.475 168.725) (size 0.8) (drill 0.3) (layers "F.Cu" "B.Cu") (free) (net 2))
@@
   (via (at 214.875 165.925) (size 0.8) (drill 0.3) (layers "F.Cu" "B.Cu") (free) (net 2))
   (via (at 240.8 171.2) (size 0.8) (drill 0.3) (layers "F.Cu" "B.Cu") (free) (net 2))
+  (via (at 217.8 122.8) (size 0.8) (drill 0.3) (layers "F.Cu" "B.Cu") (free) (net 2))
   (via (at 240.8 139.2) (size 0.8) (drill 0.3) (layers "F.Cu" "B.Cu") (free) (net 2))
+  (via (at 201.8 122.8) (size 0.8) (drill 0.3) (layers "F.Cu" "B.Cu") (free) (net 2))
+  (via (at 198.8 119.2) (size 0.8) (drill 0.3) (layers "F.Cu" "B.Cu") (free) (net 2))
+  (via (at 197.8 120.2) (size 0.8) (drill 0.3) (layers "F.Cu" "B.Cu") (free) (net 2))
   (via (at 239.8 140.2) (size 0.8) (drill 0.3) (layers "F.Cu" "B.Cu") (free) (net 2))
+  (via (at 200.8 119.2) (size 0.8) (drill 0.3) (layers "F.Cu" "B.Cu") (free) (net 2))
   (via (at 222.475 171.725) (size 0.8) (drill 0.3) (layers "F.Cu" "B.Cu") (free) (net 2))
   (via (at 238.8 157.2) (size 0.8) (drill 0.3) (layers "F.Cu" "B.Cu") (free) (net 2))
@@
   (via (at 225.55 137.2625) (size 0.8) (drill 0.3) (layers "F.Cu" "B.Cu") (free) (net 2))
   (via (at 240.8 168.2) (size 0.8) (drill 0.3) (layers "F.Cu" "B.Cu") (free) (net 2))
+  (via (at 216.8 122.8) (size 0.8) (drill 0.3) (layers "F.Cu" "B.Cu") (free) (net 2))
+  (via (at 199.8 122.8) (size 0.8) (drill 0.3) (layers "F.Cu" "B.Cu") (free) (net 2))
+  (via (at 215.8 120.2) (size 0.8) (drill 0.3) (layers "F.Cu" "B.Cu") (free) (net 2))
+  (via (at 197.8 119.2) (size 0.8) (drill 0.3) (layers "F.Cu" "B.Cu") (free) (net 2))
+  (via (at 201.8 119.2) (size 0.8) (drill 0.3) (layers "F.Cu" "B.Cu") (free) (net 2))
   (via (at 224.475 170.725) (size 0.8) (drill 0.3) (layers "F.Cu" "B.Cu") (free) (net 2))
   (via (at 226.475 170.725) (size 0.8) (drill 0.3) (layers "F.Cu" "B.Cu") (free) (net 2))
   (via (at 220.15 165.2625) (size 0.8) (drill 0.3) (layers "F.Cu" "B.Cu") (net 2))
+  (via (at 219.8 120.2) (size 0.8) (drill 0.3) (layers "F.Cu" "B.Cu") (free) (net 2))
   (via (at 227.475 171.725) (size 0.8) (drill 0.3) (layers "F.Cu" "B.Cu") (free) (net 2))
   (via (at 227.55 137.2625) (size 0.8) (drill 0.3) (layers "F.Cu" "B.Cu") (free) (net 2))
+  (via (at 218.8 119.2) (size 0.8) (drill 0.3) (layers "F.Cu" "B.Cu") (free) (net 2))
   (via (at 226.475 171.725) (size 0.8) (drill 0.3) (layers "F.Cu" "B.Cu") (free) (net 2))
   (via (at 222.475 170.725) (size 0.8) (drill 0.3) (layers "F.Cu" "B.Cu") (free) (net 2))
   (via (at 215.575 166.825) (size 0.8) (drill 0.3) (layers "F.Cu" "B.Cu") (free) (net 2))
+  (via (at 198.8 122.8) (size 0.8) (drill 0.3) (layers "F.Cu" "B.Cu") (free) (net 2))
   (via (at 216.5 189) (size 0.8) (drill 0.3) (layers "F.Cu" "B.Cu") (net 3))
   (segment (start 209.55 186.9) (end 211.675 189.025) (width 0.5) (layer "B.Cu") (net 3))
@@
         (xy 241.5 130.6)
         (xy 241.5 118)
+        (xy 241.4 118)
         (xy 232.6 118)
         (xy 232.6 118)
-        (xy 218.7 118)
         (xy 209 118)
         (xy 209 110)

Commit message: Few kicker routing change
Parts:
- J5, Q4, R1, R41: moved to B.Cu
- moved R44 208.5 mm to (233.7, 226.1)
- moved R43 194.8 mm to (248.9, 200.7), turned to 180 degrees
- moved D3 193.5 mm to (228.6, 233.7)
- moved R45 182.9 mm to (235.4, 198.1)
- moved C34 177.9 mm to (226.1, 198.1)
- moved C32 172.8 mm to (195.6, 208.3)
- moved L4 171.9 mm to (195.6, 213.4)
- moved C33 171.8 mm to (198.1, 218.4)
- moved D6 169.9 mm to (223.5, 205.7)
- moved R18 156.8 mm to (230.9, 175.8), turned to 180 degrees
- moved Q4 149.9 mm to (205.7, 175.3), turned to 180 degrees
- moved JP3 135.3 mm to (160.0, 180.3)
- moved R1 134.3 mm to (184.6, 185.4), turned to 180 degrees
- moved R16 131.6 mm to (208.7, 171.5), turned to -90 degrees
- moved R41 122.0 mm to (208.3, 172.7)
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Routing:
- net /digital/NRST: track 0.00 -> 13.2 mm, vias 0 -> 1
- net /digital/SWDIO: track 0.00 -> 5.84 mm, vias 0 -> 1
- net /digital/SWDCLK: track 0.00 -> 4.28 mm, vias 0 -> 1
- net /digital/DOTSTAR_MOSI: track 13.9 -> 11.8 mm
- net /digital/DOTSTAR_SCK: track 14.4 -> 13.9 mm
- net GND: track 21.5 -> 21.4 mm, vias 140 -> 141
- net +5V: vias 1 -> 0
