File: robot/kicker/v1.1.0/kicker/flyback_charger.kicad_sch (KiCad schematic)
At the start: 45 parts, among them Q1 BSC0402NSATMA1, U4 LT3751-QFN

Commit message: address initial issues with v1.0.0
Parts:
- JP2: footprint Jumper:SolderJumper-2_P1.3mm_Bridged_RoundedPad1.0x1.5mm -> AT-BoardFeatures:SolderJumper-2_2.0x1.2mm_Closed
- R31, R32, R33: now not fitted
Other:
- note removed: "DNP - TEST ONLY"
