File: robot/breakbeam/v1.0.0/breakbeam-emitter/breakbeam-emitter.kicad_pcb (KiCad board)
At the start: 2 copper layers, 6 parts, among them J1 Conn_01x03, Q1 RUC002N05T116

Commit message: Mechanical iteration, electrical review
Parts:
- added G***: LOGO, AT-Style:logo_3_mm_3_mm, B.Cu at (135.5, 60.5)
- added H1: MountingHole, MountingHole:MountingHole_2.2mm_M2, F.Cu at (122.0, 68.0)
- added H2: MountingHole, MountingHole:MountingHole_2.2mm_M2, F.Cu at (122.0, 59.0)
- D1: moved to B.Cu
- R1: value 43 -> 36
- moved Q1 33.5 mm to (128.0, 59.0)
- moved D1 30.1 mm to (123.3, 63.5), turned to 180 degrees
- moved J1 27.7 mm to (135.0, 63.5), turned to 90 degrees
- moved R3 23.3 mm to (126.4, 65.5), turned to 180 degrees
- moved R2 23.1 mm to (129.8, 63.6), turned to 90 degrees
- moved R1 21.9 mm to (126.4, 61.9)
Routing:
- net +3.3V: track 0.00 -> 14.4 mm
- net GND: track 0.00 -> 9.33 mm
- net Net-(Q1-G): track 0.00 -> 7.31 mm
- net BALL_TX: track 0.00 -> 6.52 mm
- net Net-(D1-K): track 0.00 -> 2.88 mm
- net Net-(Q1-D): track 0.00 -> 1.92 mm
Other:
- board outline added: 20 x 13 mm
- copper layers 2 -> 4
- board text added: "A-TEAM Breakbeam TX"
- board text added: "v1.0"
- board text added: "v1.0 5-2023"

Commit message: Ordering changes
Other:
- copper layers 4 -> 2
Changed lines of the file:
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@@
   (layers
     (0 "F.Cu" signal)
-    (1 "In1.Cu" signal)
-    (2 "In2.Cu" signal)
     (31 "B.Cu" signal)
     (32 "B.Adhes" user "B.Adhesive")
@@
       (layer "F.Mask" (type "Top Solder Mask") (color "Green") (thickness 0.01))
       (layer "F.Cu" (type "copper") (thickness 0.035))
-      (layer "dielectric 1" (type "prepreg") (thickness 0.2) (material "FR4") (epsilon_r 4.5) (loss_tangent 0.02))
-      (layer "In1.Cu" (type "copper") (thickness 0.0175))
-      (layer "dielectric 2" (type "core") (thickness 1.065) (material "FR4") (epsilon_r 4.5) (loss_tangent 0.02))
-      (layer "In2.Cu" (type "copper") (thickness 0.0175))
-      (layer "dielectric 3" (type "prepreg") (thickness 0.2) (material "FR4") (epsilon_r 4.5) (loss_tangent 0.02))
+      (layer "dielectric 1" (type "core") (thickness 1.5) (material "FR4") (epsilon_r 4.5) (loss_tangent 0.02))
       (layer "B.Cu" (type "copper") (thickness 0.035))
       (layer "B.Mask" (type "Bottom Solder Mask") (color "Green") (thickness 0.01))
@@
       (plot_on_all_layers_selection 0x0000000_00000000)
       (disableapertmacros false)
-      (usegerberextensions false)
+      (usegerberextensions true)
       (usegerberattributes true)
-      (usegerberadvancedattributes true)
-      (creategerberjobfile true)
+      (usegerberadvancedattributes false)
+      (creategerberjobfile false)
       (dashed_line_dash_ratio 12.000000)
       (dashed_line_gap_ratio 3.000000)
@@
       (psa4output false)
       (plotreference true)
-      (plotvalue true)
+      (plotvalue false)
       (plotinvisibletext false)
       (sketchpadsonfab false)
-      (subtractmaskfromsilk false)
+      (subtractmaskfromsilk true)
       (outputformat 1)
       (mirror false)
-      (drillshape 1)
+      (drillshape 0)
       (scaleselection 1)
-      (outputdirectory "")
+      (outputdirectory "breakbeam-emitter-manufacture/")
     )
   )
@@
     (pad "3" smd roundrect (at 1 -2 90) (size 0.6 1.55) (layers "F.Cu" "F.Paste" "F.Mask") (roundrect_rratio 0.25)
       (net 4 "GND") (pinfunction "Pin_3") (pintype "passive"))
-    (pad "MP" smd roundrect (at -2.3 1.875 90) (size 1.2 1.8) (layers "F.Cu" "F.Paste" "F.Mask") (roundrect_rratio 0.208333))
-    (pad "MP" smd roundrect (at 2.3 1.875 90) (size 1.2 1.8) (layers "F.Cu" "F.Paste" "F.Mask") (roundrect_rratio 0.208333))
+    (pad "MP" smd roundrect (at -2.3 1.875 90) (size 1.2 1.8) (layers "F.Cu" "F.Paste" "F.Mask") (roundrect_rratio 0.2083333333))
+    (pad "MP" smd roundrect (at 2.3 1.875 90) (size 1.2 1.8) (layers "F.Cu" "F.Paste" "F.Mask") (roundrect_rratio 0.2083333333))
     (model "C:/Users/jspal/GitHub/electrical/robot/breakbeam/v1.0.0/SM03B-SRSS-TB_LF__SN_.step"
       (offset (xyz 0 1.4 -0.24))
