File: robot/kicker/v3.0/kicker/digital.kicad_sch (KiCad schematic)
At the start: 1 part, among them U9 STM32F411RETx

Commit message: kicker v3.0 digital schematic work
Parts:
- added C48: 4u7 50V, Capacitor_SMD:C_0805_2012Metric, symbol Device:C
- added C49, C50: 0.1u, Capacitor_SMD:C_0603_1608Metric, symbol Device:C
- added D13: Blue, AT-LED:LED0603, symbol Device:LED
- added D14: Green, AT-LED:LED0603, symbol Device:LED
- added D15: Yellow, AT-LED:LED0603, symbol Device:LED
- added J4: Conn_01x10, symbol Connector_Generic:Conn_01x10
- added J7: Conn_ARM_JTAG_SWD_10, AT-Connectors:Samtec-2x5pin-0.5mm, symbol Connector:Conn_ARM_JTAG_SWD_10
- added JP7: Disable Micro, AT-BoardFeatures:SolderJumper-2_2.0x1.2mm_Open, symbol Jumper:SolderJumper_2_Open
- added Q7: BSS138K, Package_TO_SOT_SMD:SOT-23, symbol Device:Q_NMOS_GSD
- added R54, R55, R60: 10k, Resistor_SMD:R_0603_1608Metric, symbol Device:R_Small_US
- added R61: 100k, Resistor_SMD:R_0603_1608Metric, symbol Device:R_US
- added R62: 10k, symbol Device:R_Small_US
- added SW1: RST, symbol Switch:SW_Push
- added SW1: BTN0, symbol Switch:SW_Push
- added SW4: SW_DIP_x04, symbol Switch:SW_DIP_x04
- added U10, U11: SK9822, AT-LED:SK9822, symbol AT-LED:SK9822
Connections:
- net BB_RX is gone; now on net BB_{RX}: U9.24 (PC4)
- net BB_TX is gone; now on net BB_{TX}: U9.61 (PB8)
- net CMD_CHG is gone; now on net CMD_{HV_CHG}: U9.28 (PB2)
- net CMD_CHIP is gone; now on net CMD_{HV_CHIP}: U9.27 (PB1)
- net CMD_KICK is gone; now on net CMD_{HV_KICK}: U9.26 (PB0)
- net PWR_BTN_~{INT} is gone; now on net PWR_BTN_PRESSED_~{INT}: U9.56 (PB4)
- net V_{SENSE}_12v0 is gone; now on net V_{sense}_12v0: U9.9 (PC1)
- net V_{SENSE}_5v0 is gone; now on net V_{sense}_5v0: U9.10 (PC2)
- net V_{SENSE}_6v2 is gone; now on net V_{sense}_SERVO: U9.11 (PC3)
- net V_{SENSE}_HV is gone; now on net V_{sense}_HV: U9.8 (PC0)
- net BB_LED_BLUE: now also R54.1
- net BOOT_UART.BOOT0: now also Q7.1 (G), R61.1
- net DOTSTAR_MOSI: now also U10.1 (SDI)
- net DOTSTAR_SCK: now also U10.2 (CKI)
- net FLASH_MISO: now also J4.7 (Pin_7)
- net FLASH_MOSI: now also J4.8 (Pin_8)
- net FLASH_SCK: now also J4.6 (Pin_6)
- net LED_GREEN: now also R55.1
- net LED_RED: now also R60.1
- net NRST: now also C49.1, J7.10 (~{RESET}), JP7.2 (B), Q7.3 (D), SW1.2
- net SERVO_LIM1: now also J4.9 (Pin_9)
- net SERVO_LIM2: now also J4.10 (Pin_10)
- net SERVO_SS: now also J4.5 (Pin_5)
- net SWDIO: now also J7.2 (SWDIO/TMS)
- net USR_BTN: now also C50.1, R62.1, SW1.1
- net SENSE_UART.~{DET}: now reaches U9.4 (PC15)
- net DRIB_UART.~{DET}: now reaches U9.50 (PA15)
- net BB_SCL renamed BB_BUS.SCL
- net BB_SDA renamed BB_BUS.SDA
- net BSENSE_BOOT0 renamed SENSE_UART.BOOT0
- net BSENSE_RST renamed SENSE_UART.~{RST}
- net BSENSE_RX renamed SENSE_UART.RX
- net BSENSE_TX renamed SENSE_UART.TX
- net DRIB_BOOT0 renamed DRIB_UART.BOOT0
- net DRIB_RST renamed DRIB_UART.~{RST}
- net DRIB_RX renamed DRIB_UART.RX
- net DRIB_TX renamed DRIB_UART.TX
- new net: U10.6 (SDO), U11.1 (SDI)
- new net: U10.5 (CKO), U11.2 (CKI)
- new net: D14.2 (A), R55.2
- new net: D15.2 (A), R60.2
- new net: D13.2 (A), R54.2
- new net +3.3V: J4.2 (Pin_2), J7.1 (VTref), SW1.2
- new net +5V: C48.2, J4.3 (Pin_3), U10.4 (VCC), U11.4 (VCC)
- new net +6V: J4.4 (Pin_4)
- new net GND: C48.1, C49.2, C50.2, D13.1 (K), D14.1 (K), D15.1 (K), J4.1 (Pin_1), J7.3 (GND), J7.5 (GND), J7.9 (GNDDetect), JP7.1 (A), Q7.2 (S), R61.2, R62.2, SW1.1, U10.3 (GND), U11.3 (GND)
- new net SWDCLK: J7.4 (SWDCLK/TCK)
- no-connect marks 6 -> 8
Other:
- note added: "Charge Level"
- note added: "Debug Header"
- note added: "Software Indicators"
- note added: "Status"

Commit message: lots of ERC work
Parts:
- added R37, R38, R39, R40: 10k, symbol Device:R_Small_US
- renumbered C49 to C22, C50 to C23, C48 to C24, D15 to D10, D13 to D8, D14 to D9, J7 to J2, Q7 to Q4, R61 to R33, R62 to R34, R54 to R35, R55 to R36, R60 to R41, U9 to U4, U10 to U5, U11 to U6
Connections:
- net +3.3V is gone; now on net +3V3: J2.1 (VTref), J4.2 (Pin_2), SW1.2
- net SWDCLK is gone; now on net SWCLK: J2.4 (SWDCLK/TCK)
- net DIP0: now also SW4.1, R40.2
- net DIP1: now also SW4.2, R39.2
- net DIP2: now also SW4.3, R38.2
- net DIP3: now also SW4.4, R37.2
- net GND: now also SW4.5, SW4.6, SW4.7, SW4.8, U4.12 (VSSA), U4.18 (VSS), U4.31 (VSS), U4.47 (VSS), U4.63 (VSS)
- net +3V3: now reaches U4.19 (VDD)
- net +3V3: now also U4.32 (VDD), U4.48 (VDD), U4.64 (VDD), R37.1, R38.1, R39.1, R40.1
- net BB_{RX} renamed BB_BUS.BB_{RX}
- net BB_{TX} renamed BB_BUS.BB_{TX}
- net BOOT_UART.BOOT0 renamed MCU_BOOT_UART.~{RST}
- net MCU_BOOT_UART.~{RST}: no longer U4.60 (BOOT0)
- net BOOT_UART.RX renamed MCU_BOOT_UART.RX
- net BOOT_UART.TX renamed MCU_BOOT_UART.TX
- net CMD_{HV_CHG} renamed CMD_{CHG}
- net CMD_{HV_CHIP} renamed CMD_{CHIP}
- net CMD_{HV_KICK} renamed CMD_{KICK}
- new net MCU_BOOT_UART.BOOT0: U4.60 (BOOT0)
Other:
- moved on the sheet: C22, JP7, Q4, R33, SW1

Commit message: kicker v3.0 passing ERC
Parts:
- added C52: 100n 6.3V, Capacitor_SMD:C_0402_1005Metric, symbol Device:C
- added C53: 100n 10V, Capacitor_SMD:C_0402_1005Metric, symbol Device:C
- added C54: 1u 10V, Capacitor_SMD:C_0603_1608Metric, symbol Device:C
- added C55, C56: 4u7 6.3V, Capacitor_SMD:C_0402_1005Metric, symbol Device:C
- added C57, C58, C59, C60, C61, C65: 100n 6.3V, Capacitor_SMD:C_0603_1608Metric, symbol Device:C
- added C62, C63: 10n 6.3V, Capacitor_SMD:C_0603_1608Metric, symbol Device:C
- added C64: 10u 6.3V, Capacitor_SMD:C_0402_1005Metric, symbol Device:C
- added J12: Conn_01x02, symbol Connector_Generic:Conn_01x02
- added L7: 650 @100MHz, Resistor_SMD:R_0603_1608Metric, symbol Device:L_Ferrite
- added R67, R68: 10k, Resistor_SMD:R_0603_1608Metric, symbol Device:R_US
- added R69: 1M, Resistor_SMD:R_0603_1608Metric, symbol Device:R_US
- added U12: AT25DF041x-UxN-x, Package_CSP:WLCSP-8_1.58x1.63x0.35mm_Layout3x5_P0.35x0.4mm_Ball0.25mm_Pad0.25mm_NSMD, symbol Memory_Flash:AT25DF041x-UxN-x
- added U13: AD8494, Package_SO:MSOP-8_3x3mm_P0.65mm, symbol Sensor_Temperature:AD8494
- C24: value 4u7 50V -> 4u7 6.3V; footprint Capacitor_SMD:C_0805_2012Metric -> Capacitor_SMD:C_0402_1005Metric
Connections:
- net +3V3: now also U4.1 (VBAT), C52.2, C56.2, C57.1, C58.1, C59.1, C60.1, C64.2, C65.1, L7.1, U12.A1 (VCC), U12.C1 (~{HOLD}), U12.E3 (~{WP}), U13.7 (+Vs)
- net FLASH_MISO: now also U12.C3 (SO/IO1)
- net FLASH_MOSI: now also U12.D2 (SI/IO0)
- net FLASH_SCK: now also U12.E1 (SCK)
- net FLASH_SS: now also U12.A3 (~{CS})
- net GND: now also C52.1, C53.2, C54.2, C55.1, C56.1, C57.2, C58.2, C59.2, C60.2, C62.2, C63.1, C64.1, C65.2, R69.1, U12.B2 (GND), U13.2 (REF), U13.3 (-Vs)
- net LED_GREEN: now also U4.54 (PD2); no longer U4.3 (PC14)
- net SENSE_UART.~{DET}: now also U4.52 (PC11); no longer U4.4 (PC15)
- net TEMP_PROBE: now also U13.5 (SENSE), U13.6
- net at U4.13 (VDDA): now also C53.1, C54.1, L7.2
- net BB_BUS.RST: now reaches U4.29 (PB10)
- net at U4.30 (VCAP1): now also C55.2
- net OSC_IN renamed 8MHZ_CLK_REF
- new net: C61.2, C62.1, R68.2, U13.8 (+IN)
- new net: J12.1 (Pin_1), R67.1, R69.2
- new net: C61.1, C63.2, R67.2, U13.1 (-IN)
- new net: J12.2 (Pin_2), R68.1
- new net 32KHZ_CLK_REF: U4.3 (PC14)
- no-connect marks 8 -> 6
Other:
- note removed: "DOTSTAR_MISO"
- company: (none) -> SSL A-Team
- title: (none) -> Kicker v3.0
- moved on the sheet: C22, C23, C24, D10, D8, D9, J2, J4, JP7, Q4, R33, R34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

Commit message: footprint work
Parts:
- C22, C23: value 0.1u -> 100n 6.3V; footprint Capacitor_SMD:C_0603_1608Metric -> (none)
- C24, C55, C56: value 4u7 6.3V -> 4.7u 6.3V; footprint Capacitor_SMD:C_0402_1005Metric -> (none)
- C52, C64: footprint Capacitor_SMD:C_0402_1005Metric -> (none)
- C53: value 100n 10V -> 100n 6.3V; footprint Capacitor_SMD:C_0402_1005Metric -> (none)
- C54: value 1u 10V -> 1u 6.3V; footprint Capacitor_SMD:C_0603_1608Metric -> (none)
- C57, C58, C59, C60, C61, C62, C63, C65: footprint Capacitor_SMD:C_0603_1608Metric -> (none)
- J4: footprint (none) -> Connector_JST:JST_SH_SM10B-SRSS-TB_1x10-1MP_P1.00mm_Horizontal
- R33, R35, R36, R41, R67, R68, R69: footprint Resistor_SMD:R_0603_1608Metric -> Resistor_SMD:R_0402_1005Metric
- R34, R37, R38, R39, R40: footprint (none) -> Resistor_SMD:R_0402_1005Metric
Other:
- moved on the sheet: C54

Commit message: kicker v3.0 footprint work
Parts:
- C22, C23, C24, C52, C53, C54, C55, C56, C57, C58, C59, C60, C61, C62, C63, C64, C65: footprint (none) -> Capacitor_SMD:C_0402_1005Metric
- J12: footprint (none) -> Connector_JST:JST_SH_SM02B-SRSS-TB_1x02-1MP_P1.00mm_Horizontal
Changed lines of the file:
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@@
       (effects (font (size 1.27 1.27)) (justify right))
     )
-    (property "Footprint" "" (at 480.3648 44.45 0)
+    (property "Footprint" "Capacitor_SMD:C_0402_1005Metric" (at 480.3648 44.45 0)
       (effects (font (size 1.27 1.27)) hide)
     )
@@
       (effects (font (size 1.27 1.27)) (justify right))
     )
-    (property "Footprint" "" (at 86.6648 234.95 0)
+    (property "Footprint" "Capacitor_SMD:C_0402_1005Metric" (at 86.6648 234.95 0)
       (effects (font (size 1.27 1.27)) hide)
     )
@@
       (effects (font (size 1.27 1.27)) (justify right))
     )
-    (property "Footprint" "" (at 57.4548 283.21 0)
+    (property "Footprint" "Capacitor_SMD:C_0402_1005Metric" (at 57.4548 283.21 0)
       (effects (font (size 1.27 1.27)) hide)
     )
@@
       (effects (font (size 1.27 1.27)))
     )
-    (property "Footprint" "" (at 48.26 217.17 0)
+    (property "Footprint" "Connector_JST:JST_SH_SM02B-SRSS-TB_1x02-1MP_P1.00mm_Horizontal" (at 48.26 217.17 0)
       (effects (font (size 1.27 1.27)) hide)
     )
@@
       (effects (font (size 1.27 1.27)) (justify left))
     )
-    (property "Footprint" "" (at 238.4552 365.76 0)
+    (property "Footprint" "Capacitor_SMD:C_0402_1005Metric" (at 238.4552 365.76 0)
       (effects (font (size 1.27 1.27)) hide)
     )
@@
       (effects (font (size 1.27 1.27)) (justify right))
     )
-    (property "Footprint" "" (at 541.3248 237.49 0)
+    (property "Footprint" "Capacitor_SMD:C_0402_1005Metric" (at 541.3248 237.49 0)
       (effects (font (size 1.27 1.27)) hide)
     )
@@
       (effects (font (size 1.27 1.27)) (justify right))
     )
-    (property "Footprint" "" (at 322.8848 93.98 0)
+    (property "Footprint" "Capacitor_SMD:C_0402_1005Metric" (at 322.8848 93.98 0)
       (effects (font (size 1.27 1.27)) hide)
     )
@@
       (effects (font (size 1.27 1.27)) (justify right))
     )
-    (property "Footprint" "" (at 255.5748 177.8 0)
+    (property "Footprint" "Capacitor_SMD:C_0402_1005Metric" (at 255.5748 177.8 0)
       (effects (font (size 1.27 1.27)) hide)
     )
@@
       (effects (font (size 1.27 1.27)) (justify right))
     )
-    (property "Footprint" "" (at 86.6648 209.55 0)
+    (property "Footprint" "Capacitor_SMD:C_0402_1005Metric" (at 86.6648 209.55 0)
       (effects (font (size 1.27 1.27)) hide)
     )
@@
       (effects (font (size 1.27 1.27)) (justify right))
     )
-    (property "Footprint" "" (at 303.8348 93.98 0)
+    (property "Footprint" "Capacitor_SMD:C_0402_1005Metric" (at 303.8348 93.98 0)
       (effects (font (size 1.27 1.27)) hide)
     )
@@
       (effects (font (size 1.27 1.27)) (justify left))
     )
-    (property "Footprint" "" (at 479.7552 358.14 0)
+    (property "Footprint" "Capacitor_SMD:C_0402_1005Metric" (at 479.7552 358.14 0)
       (effects (font (size 1.27 1.27)) hide)
     )
@@
       (effects (font (size 1.27 1.27)) (justify right))
     )
-    (property "Footprint" "" (at 95.5548 290.83 0)
+    (property "Footprint" "Capacitor_SMD:C_0402_1005Metric" (at 95.5548 290.83 0)
       (effects (font (size 1.27 1.27)) hide)
     )
@@
       (effects (font (size 1.27 1.27)) (justify right))
     )
-    (property "Footprint" "" (at 133.6548 290.83 0)
+    (property "Footprint" "Capacitor_SMD:C_0402_1005Metric" (at 133.6548 290.83 0)
       (effects (font (size 1.27 1.27)) hide)
     )
@@
       (effects (font (size 1.27 1.27)) (justify right))
     )
-    (property "Footprint" "" (at 86.6648 222.25 0)
+    (property "Footprint" "Capacitor_SMD:C_0402_1005Metric" (at 86.6648 222.25 0)
       (effects (font (size 1.27 1.27)) hide)
     )
@@
       (effects (font (size 1.27 1.27)) (justify right))
     )
-    (property "Footprint" "" (at 131.1148 200.66 0)
+    (property "Footprint" "Capacitor_SMD:C_0402_1005Metric" (at 131.1148 200.66 0)
       (effects (font (size 1.27 1.27)) hide)
     )
@@
       (effects (font (size 1.27 1.27)) (justify right))
     )
-    (property "Footprint" "" (at 114.6048 290.83 0)
+    (property "Footprint" "Capacitor_SMD:C_0402_1005Metric" (at 114.6048 290.83 0)
       (effects (font (size 1.27 1.27)) hide)
     )
@@
       (effects (font (size 1.27 1.27)) (justify right))
     )
-    (property "Footprint" "" (at 151.4348 193.04 0)
+    (property "Footprint" "Capacitor_SMD:C_0402_1005Metric" (at 151.4348 193.04 0)
       (effects (font (size 1.27 1.27)) hide)
     )
@@
       (effects (font (size 1.27 1.27)) (justify right))
     )
-    (property "Footprint" "" (at 76.5048 290.83 0)
-      (effects (font (size 1.27 1.27)) hide)
-    )
+    (property "Footprint" "Capacitor_SMD:C_0402_1005Metric" (at 76.5048 290.83 0)
+      (effects (font (size 1.27 1.27)) hide)
+    )

Commit message: kicker v3.0 footprint work
Parts:
- SW1: footprint (none) -> Button_Switch_SMD:SW_SPST_TL3305A
- SW4: footprint (none) -> Button_Switch_SMD:SW_DIP_SPSTx04_Slide_Omron_A6S-410x_W8.9mm_P2.54mm
Other:
- note added: "Reset Logic"
Changed lines of the file:
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@@
     (stroke (width 0) (type default))
   )
-  (wire (pts (xy 57.15 60.96) (xy 49.53 60.96))
+  (wire (pts (xy 57.15 55.88) (xy 49.53 55.88))
     (stroke (width 0) (type default))
   )
@@
     (stroke (width 0) (type default))
   )
-  (wire (pts (xy 57.15 66.04) (xy 49.53 66.04))
+  (wire (pts (xy 57.15 60.96) (xy 49.53 60.96))
     (stroke (width 0) (type default))
   )
@@
     (stroke (width 0) (type default))
   )
-  (wire (pts (xy 49.53 54.61) (xy 57.15 54.61))
+  (wire (pts (xy 49.53 49.53) (xy 57.15 49.53))
     (stroke (width 0) (type default))
   )
@@
     (stroke (width 0) (type default))
   )
-  (wire (pts (xy 49.53 49.53) (xy 57.15 49.53))
+  (wire (pts (xy 49.53 44.45) (xy 57.15 44.45))
     (stroke (width 0) (type default))
   )
@@
     (stroke (width 0) (type default))
   )
-  (wire (pts (xy 49.53 44.45) (xy 57.15 44.45))
+  (wire (pts (xy 49.53 39.37) (xy 57.15 39.37))
     (stroke (width 0) (type default))
   )
@@
     (stroke (width 0) (type default))
   )
-  (wire (pts (xy 49.53 41.91) (xy 57.15 41.91))
+  (wire (pts (xy 49.53 36.83) (xy 57.15 36.83))
     (stroke (width 0) (type default))
   )
@@
     (stroke (width 0) (type default))
   )
-  (wire (pts (xy 49.53 52.07) (xy 57.15 52.07))
+  (wire (pts (xy 49.53 46.99) (xy 57.15 46.99))
     (stroke (width 0) (type default))
   )
@@
     (stroke (width 0) (type default))
   )
-  (wire (pts (xy 57.15 63.5) (xy 49.53 63.5))
+  (wire (pts (xy 57.15 58.42) (xy 49.53 58.42))
     (stroke (width 0) (type default))
   )
@@
     (stroke (width 0) (type default))
   )
-  (wire (pts (xy 57.15 68.58) (xy 49.53 68.58))
+  (wire (pts (xy 57.15 63.5) (xy 49.53 63.5))
     (stroke (width 0) (type default))
   )
@@
     (stroke (width 0) (type default))
   )
+  (rectangle (start 101.6 334.01) (end 264.16 401.32)
+    (stroke (width 0) (type default))
+    (fill (type none))
+  )
+  (rectangle (start 20.32 20.32) (end 86.36 69.85)
+    (stroke (width 0) (type default))
+    (fill (type none))
+  )
   (text "Debug Header" (at 20.32 336.55 0)
     (effects (font (size 1.27 1.27)) (justify left bottom))
@@
     (effects (font (size 1.27 1.27)) (justify left bottom))
   )
+  (text "Reset Logic" (at 102.87 337.82 0)
+    (effects (font (size 1.27 1.27)) (justify left bottom))
+  )
   (text "Software Indicators" (at 470.535 21.59 0)
     (effects (font (size 1.27 1.27)) (justify left bottom))
@@
     (effects (font (size 1.27 1.27)) (justify right bottom))
   )
-  (label "PWR_BTN_PRESSED_~{INT}" (at 57.15 41.91 0) (fields_autoplaced)
+  (label "PWR_BTN_PRESSED_~{INT}" (at 57.15 36.83 0) (fields_autoplaced)
     (effects (font (size 1.27 1.27)) (justify left bottom))
   )
@@
     (effects (font (size 1.27 1.27)) (justify right bottom))
   )
-  (label "CMD_{CHIP}" (at 57.15 52.07 0) (fields_autoplaced)
+  (label "CMD_{CHIP}" (at 57.15 46.99 0) (fields_autoplaced)
     (effects (font (size 1.27 1.27)) (justify left bottom))
   )
@@
     (effects (font (size 1.27 1.27)) (justify right bottom))
   )
-  (label "V_{sense}_6v2" (at 57.15 68.58 0) (fields_autoplaced)
+  (label "V_{sense}_6v2" (at 57.15 63.5 0) (fields_autoplaced)
     (effects (font (size 1.27 1.27)) (justify left bottom))
   )
@@
     (effects (font (size 1.27 1.27)) (justify left bottom))
   )
-  (label "PWR_KILL" (at 57.15 44.45 0) (fields_autoplaced)
+  (label "PWR_KILL" (at 57.15 39.37 0) (fields_autoplaced)
     (effects (font (size 1.27 1.27)) (justify left bottom))
   )
@@
     (effects (font (size 1.27 1.27)) (justify right bottom))
   )
-  (label "V_{sense}_12v0" (at 57.15 63.5 0) (fields_autoplaced)
+  (label "V_{sense}_12v0" (at 57.15 58.42 0) (fields_autoplaced)
     (effects (font (size 1.27 1.27)) (justify left bottom))
   )
@@
     (effects (font (size 1.27 1.27)) (justify left bottom))
   )
-  (label "CMD_{CHG}" (at 57.15 54.61 0) (fields_autoplaced)
+  (label "CMD_{CHG}" (at 57.15 49.53 0) (fields_autoplaced)
     (effects (font (size 1.27 1.27)) (justify left bottom))
   )
@@
     (effects (font (size 1.27 1.27)) (justify left bottom))
   )
-  (label "V_{sense}_HV" (at 57.15 60.96 0) (fields_autoplaced)
+  (label "V_{sense}_HV" (at 57.15 55.88 0) (fields_autoplaced)
     (effects (font (size 1.27 1.27)) (justify left bottom))
   )
@@
     (effects (font (size 1.27 1.27)) (justify right bottom))
   )
-  (label "CMD_{KICK}" (at 57.15 49.53 0) (fields_autoplaced)
+  (label "CMD_{KICK}" (at 57.15 44.45 0) (fields_autoplaced)
     (effects (font (size 1.27 1.27)) (justify left bottom))
   )
@@
     (effects (font (size 1.27 1.27)) (justify left bottom))
   )
-  (label "V_{sense}_5v0" (at 57.15 66.04 0) (fields_autoplaced)
+  (label "V_{sense}_5v0" (at 57.15 60.96 0) (fields_autoplaced)
     (effects (font (size 1.27 1.27)) (justify left bottom))
   )
@@
     (effects (font (size 1.27 1.27)) (justify right))
   )
-  (hierarchical_label "PWR_BTN_PRESSED_~{INT}" (shape input) (at 49.53 41.91 180) (fields_autoplaced)
+  (hierarchical_label "PWR_BTN_PRESSED_~{INT}" (shape input) (at 49.53 36.83 180) (fields_autoplaced)
     (effects (font (size 1.27 1.27)) (justify right))
   )
-  (hierarchical_label "V_{sense}_5v0" (shape input) (at 49.53 66.04 180) (fields_autoplaced)
+  (hierarchical_label "V_{sense}_5v0" (shape input) (at 49.53 60.96 180) (fields_autoplaced)
     (effects (font (size 1.27 1.27)) (justify right))
   )
-  (hierarchical_label "CMD_{CHG}" (shape output) (at 49.53 54.61 180) (fields_autoplaced)
+  (hierarchical_label "CMD_{CHG}" (shape output) (at 49.53 49.53 180) (fields_autoplaced)
     (effects (font (size 1.27 1.27)) (justify right))
   )
@@
     (effects (font (size 1.27 1.27)) (justify right))
   )
-  (hierarchical_label "CMD_{KICK}" (shape output) (at 49.53 49.53 180) (fields_autoplaced)
+  (hierarchical_label "CMD_{KICK}" (shape output) (at 49.53 44.45 180) (fields_autoplaced)
     (effects (font (size 1.27 1.27)) (justify right))
   )
-  (hierarchical_label "V_{sense}_12v0" (shape input) (at 49.53 63.5 180) (fields_autoplaced)
+  (hierarchical_label "V_{sense}_12v0" (shape input) (at 49.53 58.42 180) (fields_autoplaced)
     (effects (font (size 1.27 1.27)) (justify right))
   )
@@
     (effects (font (size 1.27 1.27)) (justify left))
   )
-  (hierarchical_label "PWR_KILL" (shape output) (at 49.53 44.45 180) (fields_autoplaced)
+  (hierarchical_label "PWR_KILL" (shape output) (at 49.53 39.37 180) (fields_autoplaced)
     (effects (font (size 1.27 1.27)) (justify right))
   )
-  (hierarchical_label "V_{sense}_HV" (shape input) (at 49.53 60.96 180) (fields_autoplaced)
+  (hierarchical_label "V_{sense}_HV" (shape input) (at 49.53 55.88 180) (fields_autoplaced)
     (effects (font (size 1.27 1.27)) (justify right))
   )
@@
     (effects (font (size 1.27 1.27)) (justify right))
   )
-  (hierarchical_label "CMD_{CHIP}" (shape output) (at 49.53 52.07 180) (fields_autoplaced)
+  (hierarchical_label "CMD_{CHIP}" (shape output) (at 49.53 46.99 180) (fields_autoplaced)
     (effects (font (size 1.27 1.27)) (justify right))
   )
@@
     (effects (font (size 1.27 1.27)) (justify left))
   )
-  (hierarchical_label "V_{sense}_SERVO" (shape input) (at 49.53 68.58 180) (fields_autoplaced)
+  (hierarchical_label "V_{sense}_SERVO" (shape input) (at 49.53 63.5 180) (fields_autoplaced)
     (effects (font (size 1.27 1.27)) (justify right))
   )
@@
       (effects (font (size 1.27 1.27)) (justify left))
     )
-    (property "Footprint" "" (at 530.86 344.17 0)
+    (property "Footprint" "Button_Switch_SMD:SW_DIP_SPSTx04_Slide_Omron_A6S-410x_W8.9mm_P2.54mm" (at 530.86 344.17 0)
       (effects (font (size 1.27 1.27)) hide)
     )
@@
       (effects (font (size 1.27 1.27)) (justify right))
     )
-    (property "Footprint" "" (at 191.77 363.22 0)
+    (property "Footprint" "Button_Switch_SMD:SW_SPST_TL3305A" (at 191.77 363.22 0)
       (effects (font (size 1.27 1.27)) hide)
     )
@@
       (effects (font (size 1.27 1.27)) (justify right))
     )
-    (property "Footprint" "" (at 454.66 335.28 0)
+    (property "Footprint" "Button_Switch_SMD:SW_SPST_TL3305A" (at 454.66 335.28 0)
       (effects (font (size 1.27 1.27)) hide)
     )

Commit message: kicker v3.0 ready for review
Other:
- note added: "Flash Chip"
- note added: "H to L Nets"
- note added: "Microcontroller"
- note added: "Servo/SPI Aux Connector"
- note added: "Temp Sensing"
- note added: "User Button"
- note added: "User DIP SW"
- note added: "uC Decoupling"
- moved on the sheet: C22, C23, C24, C52, C53, C54, C55, C56, C57, C58, C59, C60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
