File: robot/kicker/v3.0/kicker/hv_kicker.kicad_sch (KiCad schematic)
At the start: 0 parts

Commit message: kicker work
Parts:
- added C22, C23, C24: 1000uF 200V, AT-Capacitors:ESMQ201VSN102MQ35S, symbol Device:C_Polarized
- added D8, D9: RED, AT-LED:LED0603, symbol Device:LED
- added R26, R27, R28, R29: 1M47, Resistor_SMD:R_0603_1608Metric, symbol Device:R_US
- added R30, R31: 475k, Resistor_SMD:R_0603_1608Metric, symbol Device:R_US
- added R32: 4k75, Resistor_SMD:R_0603_1608Metric, symbol Device:R_US
Connections:
- net HV_MON: now also R31.2, R32.1
- new net: D8.2 (A), R27.2
- new net: D9.2 (A), R29.2
- new net DL1S: R26.2, R27.1
- new net DL2S: R28.2, R29.1
- new net GND: C22.2, C23.2, C24.2, D8.1 (K), D9.1 (K), R32.2
- new net HVMS: R30.2, R31.1
- new net flyback_charger/V_{solenoid}: C22.1, C23.1, C24.1, R26.1, R28.1, R30.1
Other:
- added sheet flyback_charger (flyback_charger.kicad_sch)
- added sheet solenoid_control (solenoid_control.kicad_sch)
- note added: "0.995V ref at 200V rail"
- note added: "DEATHLIGHT"
- note added: "Energy Bank"
- note added: "Solenoid Impulse Circuit"

Commit message: lots of ERC work
Parts:
- renumbered C22 to C25, C23 to C26, C24 to C27, D8 to D11, D9 to D12, R26 to R42, R27 to R43, R28 to R44, R29 to R45, R30 to R46, R31 to R47, R32 to R48
Other:
- sheet flyback_charger ports: added V_{BATT}; removed V_{batt}
- sheet solenoid_control ports: added CMD_{CHIP}, CMD_{KICK}; removed CMD_{chip}, CMD_{kick}

Commit message: kicker v3.0 passing ERC
Other:
- company: (none) -> SSL A-Team
- title: (none) -> Kicker v3.0
Changed lines of the file:
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@@
 (kicad_sch (version 20230121) (generator eeschema)
   (paper "A4")
+  (title_block
+    (title "Kicker v3.0")
+    (date "2023-11-07")
+    (rev "0")
+    (company "SSL A-Team")
+    (comment 1 "Author: William Stuckey")
+  )
   (junction (at 179.07 78.74) (diameter 0) (color 0 0 0 0)
   )

Commit message: footprint work
Parts:
- D11, D12: value RED -> Red
- R42, R43, R44, R45, R46, R47, R48: footprint Resistor_SMD:R_0603_1608Metric -> Resistor_SMD:R_0402_1005Metric
Changed lines of the file:
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@@
       (effects (font (size 1.27 1.27)) (justify left))
     )
-    (property "Footprint" "Resistor_SMD:R_0603_1608Metric" (at 161.036 57.404 90)
+    (property "Footprint" "Resistor_SMD:R_0402_1005Metric" (at 161.036 57.404 90)
       (effects (font (size 1.27 1.27)) hide)
     )
@@
       (effects (font (size 1.27 1.27)) (justify right))
     )
-    (property "Value" "RED" (at 151.765 80.3274 90)
+    (property "Value" "Red" (at 151.765 80.3274 90)
       (effects (font (size 1.27 1.27)) (justify right))
     )
@@
       (effects (font (size 1.27 1.27)) (justify left))
     )
-    (property "Footprint" "Resistor_SMD:R_0603_1608Metric" (at 180.086 67.564 90)
+    (property "Footprint" "Resistor_SMD:R_0402_1005Metric" (at 180.086 67.564 90)
       (effects (font (size 1.27 1.27)) hide)
     )
@@
       (effects (font (size 1.27 1.27)) (justify left))
     )
-    (property "Footprint" "Resistor_SMD:R_0603_1608Metric" (at 180.086 89.154 90)
+    (property "Footprint" "Resistor_SMD:R_0402_1005Metric" (at 180.086 89.154 90)
       (effects (font (size 1.27 1.27)) hide)
     )
@@
       (effects (font (size 1.27 1.27)) (justify left))
     )
-    (property "Footprint" "Resistor_SMD:R_0603_1608Metric" (at 149.606 67.564 90)
+    (property "Footprint" "Resistor_SMD:R_0402_1005Metric" (at 149.606 67.564 90)
       (effects (font (size 1.27 1.27)) hide)
     )
@@
       (effects (font (size 1.27 1.27)) (justify left))
     )
-    (property "Footprint" "Resistor_SMD:R_0603_1608Metric" (at 180.086 57.404 90)
+    (property "Footprint" "Resistor_SMD:R_0402_1005Metric" (at 180.086 57.404 90)
       (effects (font (size 1.27 1.27)) hide)
     )
@@
       (effects (font (size 1.27 1.27)) (justify left))
     )
-    (property "Footprint" "Resistor_SMD:R_0603_1608Metric" (at 149.606 57.404 90)
+    (property "Footprint" "Resistor_SMD:R_0402_1005Metric" (at 149.606 57.404 90)
       (effects (font (size 1.27 1.27)) hide)
     )
@@
       (effects (font (size 1.27 1.27)) (justify left))
     )
-    (property "Footprint" "Resistor_SMD:R_0603_1608Metric" (at 161.036 67.564 90)
+    (property "Footprint" "Resistor_SMD:R_0402_1005Metric" (at 161.036 67.564 90)
       (effects (font (size 1.27 1.27)) hide)
     )
@@
       (effects (font (size 1.27 1.27)) (justify right))
     )
-    (property "Value" "RED" (at 163.195 80.3274 90)
+    (property "Value" "Red" (at 163.195 80.3274 90)
       (effects (font (size 1.27 1.27)) (justify right))
     )

Commit message: component/footprint swaps, layout work
Parts:
- C25, C26, C27: footprint AT-Capacitors:ESMQ201VSN102MQ35S -> Capacitor_THT:CP_Radial_D25.0mm_P10.00mm_SnapIn
Changed lines of the file:
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@@
       (effects (font (size 1.27 1.27)) (justify left))
     )
-    (property "Footprint" "AT-Capacitors:ESMQ201VSN102MQ35S" (at 106.3752 58.42 0)
+    (property "Footprint" "Capacitor_THT:CP_Radial_D25.0mm_P10.00mm_SnapIn" (at 106.3752 58.42 0)
       (effects (font (size 1.27 1.27)) hide)
     )
@@
       (effects (font (size 1.27 1.27)) (justify left))
     )
-    (property "Footprint" "AT-Capacitors:ESMQ201VSN102MQ35S" (at 126.6952 58.42 0)
+    (property "Footprint" "Capacitor_THT:CP_Radial_D25.0mm_P10.00mm_SnapIn" (at 126.6952 58.42 0)
       (effects (font (size 1.27 1.27)) hide)
     )
@@
       (effects (font (size 1.27 1.27)) (justify left))
     )
-    (property "Footprint" "AT-Capacitors:ESMQ201VSN102MQ35S" (at 116.5352 58.42 0)
-      (effects (font (size 1.27 1.27)) hide)
-    )
+    (property "Footprint" "Capacitor_THT:CP_Radial_D25.0mm_P10.00mm_SnapIn" (at 116.5352 58.42 0)
+      (effects (font (size 1.27 1.27)) hide)
+    )

Commit message: kicker v3.0 changes from design review
Parts:
- R42, R43, R44, R45, R46, R47: footprint Resistor_SMD:R_0402_1005Metric -> Resistor_SMD:R_0805_2012Metric
Changed lines of the file:
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@@
       (effects (font (size 1.27 1.27)) (justify left))
     )
-    (property "Footprint" "Resistor_SMD:R_0402_1005Metric" (at 161.036 57.404 90)
+    (property "Footprint" "Resistor_SMD:R_0805_2012Metric" (at 161.036 57.404 90)
       (effects (font (size 1.27 1.27)) hide)
     )
@@
       (effects (font (size 1.27 1.27)) (justify left))
     )
-    (property "Footprint" "Resistor_SMD:R_0402_1005Metric" (at 180.086 67.564 90)
+    (property "Footprint" "Resistor_SMD:R_0805_2012Metric" (at 180.086 67.564 90)
       (effects (font (size 1.27 1.27)) hide)
     )
@@
       (effects (font (size 1.27 1.27)) (justify left))
     )
-    (property "Footprint" "Resistor_SMD:R_0402_1005Metric" (at 149.606 67.564 90)
+    (property "Footprint" "Resistor_SMD:R_0805_2012Metric" (at 149.606 67.564 90)
       (effects (font (size 1.27 1.27)) hide)
     )
@@
       (effects (font (size 1.27 1.27)) (justify left))
     )
-    (property "Footprint" "Resistor_SMD:R_0402_1005Metric" (at 180.086 57.404 90)
+    (property "Footprint" "Resistor_SMD:R_0805_2012Metric" (at 180.086 57.404 90)
       (effects (font (size 1.27 1.27)) hide)
     )
@@
       (effects (font (size 1.27 1.27)) (justify left))
     )
-    (property "Footprint" "Resistor_SMD:R_0402_1005Metric" (at 149.606 57.404 90)
+    (property "Footprint" "Resistor_SMD:R_0805_2012Metric" (at 149.606 57.404 90)
       (effects (font (size 1.27 1.27)) hide)
     )
@@
       (effects (font (size 1.27 1.27)) (justify left))
     )
-    (property "Footprint" "Resistor_SMD:R_0402_1005Metric" (at 161.036 67.564 90)
-      (effects (font (size 1.27 1.27)) hide)
-    )
+    (property "Footprint" "Resistor_SMD:R_0805_2012Metric" (at 161.036 67.564 90)
+      (effects (font (size 1.27 1.27)) hide)
+    )

Commit message: finish schematic fixes from the design review, layout work
Parts:
- R42, R43, R44, R45: value 1M47 -> 1.47M
- R48: value 4k75 -> 4.75k
Changed lines of the file:
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@@
       (effects (font (size 1.27 1.27)) (justify left))
     )
-    (property "Value" "1M47" (at 161.925 58.4199 0)
+    (property "Value" "1.47M" (at 161.925 58.4199 0)
       (effects (font (size 1.27 1.27)) (justify left))
     )
@@
       (effects (font (size 1.27 1.27)) (justify left))
     )
-    (property "Value" "4k75" (at 181.61 90.805 0)
+    (property "Value" "4.75k" (at 181.61 90.805 0)
       (effects (font (size 1.27 1.27)) (justify left))
     )
@@
       (effects (font (size 1.27 1.27)) (justify left))
     )
-    (property "Value" "1M47" (at 150.495 68.5799 0)
+    (property "Value" "1.47M" (at 150.495 68.5799 0)
       (effects (font (size 1.27 1.27)) (justify left))
     )
@@
       (effects (font (size 1.27 1.27)) (justify left))
     )
-    (property "Value" "1M47" (at 150.495 58.4199 0)
+    (property "Value" "1.47M" (at 150.495 58.4199 0)
       (effects (font (size 1.27 1.27)) (justify left))
     )
@@
       (effects (font (size 1.27 1.27)) (justify left))
     )
-    (property "Value" "1M47" (at 161.925 68.5799 0)
-      (effects (font (size 1.27 1.27)) (justify left))
-    )
+    (property "Value" "1.47M" (at 161.925 68.5799 0)
+      (effects (font (size 1.27 1.27)) (justify left))
+    )

Commit message: kicker layout work
Parts:
- D11, D12: footprint AT-LED:LED0603 -> AT-LED:APA1606; LCSC C264440 -> C3034753
Changed lines of the file:
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@@
-    )
-  )
-  (symbol (lib_id "Device:LED") (at 148.59 77.47 90) (unit 1)
-    (in_bom yes) (on_board yes) (dnp no) (fields_autoplaced)
-    (property "Reference" "D11" (at 151.765 77.7874 90)
-      (effects (font (size 1.27 1.27)) (justify right))
-    )
-    (property "Value" "Red" (at 151.765 80.3274 90)
-      (effects (font (size 1.27 1.27)) (justify right))
-    )
-    (property "Footprint" "AT-LED:LED0603" (at 148.59 77.47 0)
-      (effects (font (size 1.27 1.27)) hide)
-    )
-    (property "Datasheet" "~" (at 148.59 77.47 0)
-      (effects (font (size 1.27 1.27)) hide)
-    )
-    (property "LCSC" "C264440" (at 151.765 77.7874 0)
-      (effects (font (size 1.27 1.27)) hide)
-    )
-    (pin "1")
-    (pin "2")
-    (instances
-      (project "kicker"
-        (path "/7c007fad-bfbf-4e78-a837-1f8089552516/7eb261a6-326a-4be1-a81a-5b1bf336a030"
-          (reference "D11") (unit 1)
-        )
-      )
-      (project "kicker"
-        (path "/7cfeeadc-5484-43a0-8ad3-94ff54fbcb4b"
-          (reference "D7") (unit 1)
-        )
-      )
     )
   )
@@
       (effects (font (size 1.27 1.27)) (justify right))
     )
-    (property "Footprint" "AT-LED:LED0603" (at 160.02 77.47 0)
-      (effects (font (size 1.27 1.27)) hide)
-    )
-    (property "Datasheet" "~" (at 160.02 77.47 0)
-      (effects (font (size 1.27 1.27)) hide)
-    )
-    (property "LCSC" "C264440" (at 163.195 77.7874 0)
+    (property "Footprint" "AT-LED:APA1606" (at 160.02 77.47 0)
+      (effects (font (size 1.27 1.27)) hide)
+    )
+    (property "Datasheet" "https://datasheet.lcsc.com/lcsc/2305112030_Kingbright-APA1606SURCK_C3034753.pdf" (at 160.02 77.47 0)
+      (effects (font (size 1.27 1.27)) hide)
+    )
+    (property "LCSC" "C3034753" (at 163.195 77.7874 0)
       (effects (font (size 1.27 1.27)) hide)
     )
@@
         )
       )
+    )
+  )
+  (symbol (lib_id "Device:LED") (at 148.59 77.47 90) (unit 1)
+    (in_bom yes) (on_board yes) (dnp no) (fields_autoplaced)
+    (property "Reference" "D11" (at 151.765 77.7874 90)
+      (effects (font (size 1.27 1.27)) (justify right))
+    )
+    (property "Value" "Red" (at 151.765 80.3274 90)
+      (effects (font (size 1.27 1.27)) (justify right))
+    )
+    (property "Footprint" "AT-LED:APA1606" (at 148.59 77.47 0)
+      (effects (font (size 1.27 1.27)) hide)
+    )
+    (property "Datasheet" "https://datasheet.lcsc.com/lcsc/2305112030_Kingbright-APA1606SURCK_C3034753.pdf" (at 148.59 77.47 0)
+      (effects (font (size 1.27 1.27)) hide)
+    )
+    (property "LCSC" "C3034753" (at 151.765 77.7874 0)
+      (effects (font (size 1.27 1.27)) hide)
+    )
+    (pin "1")
+    (pin "2")
+    (instances
+      (project "kicker"
+        (path "/7c007fad-bfbf-4e78-a837-1f8089552516/7eb261a6-326a-4be1-a81a-5b1bf336a030"
+          (reference "D11") (unit 1)
+        )
+      )
+      (project "kicker"
+        (path "/7cfeeadc-5484-43a0-8ad3-94ff54fbcb4b"
+          (reference "D8") (unit 1)
+        )
+      )
