File: robot/kicker/v3.0/kicker/kicker.kicad_pcb (KiCad board)
At the start: 4 copper layers, 113 x 110 mm, 223 parts, among them J1 XT30-F, J10 Conn_01x10, J11 Conn_01x06, J12 Conn_01x02, J13 Conn_01x02, J2 Conn_ARM_JTAG_SWD_10, J3 Conn_01x10, J4 Conn_01x10, J5 Conn_01x02, J6 Conn_01x02, J7 Conn_01x10, J8 Conn_01x03, J9 Conn_01x03, Q1 BSS138, Q2 SQJA80EP-T1_GE3, Q3 SQJA80EP-T1_GE3, Q4 BSS138K, Q5 IXGA48N60A3, Q6 IXGA48N60A3, Q7 BSC0402NSATMA1, SW1 PWR_ON, SW2 RST, SW3 BTN0, SW4 SW_DIP_x04, U1 LTC4367, U10 IX4427, U11 LT3757EMSE, U12 AT25DF041x-UxN-x, U13 AD8494, U2 LTC2955-1, U3 LT3504, U4 STM32F411RETx, U5 SK9822, U6 SK9822, U7 ISO6720-Q1, U8 ISO6721-Q1, U9 ISO6720-Q1

Commit message: lots of kicker work
Parts:
- removed Ce1: 470n 6.3V, Capacitor_SMD:C_0402_1005Metric
- removed L7: 650 @100MHz, Resistor_SMD:R_0603_1608Metric
- removed U4: STM32F411RETx, Package_QFP:LQFP-64_10x10mm_P0.5mm
- added C10: 4.7u 6.3V, Capacitor_SMD:C_0402_1005Metric, F.Cu at (-40.0, 183.6)
- added C66: 4.7u 6.3V, Capacitor_SMD:C_0402_1005Metric, F.Cu at (-40.0, 185.5)
- added C67: 100n 50V, Capacitor_SMD:C_0402_1005Metric, F.Cu at (-40.0, 187.5)
- added C68: 1u 50V, Capacitor_SMD:C_0402_1005Metric, F.Cu at (-40.0, 189.5)
- added C69: 470n 6.3V, Capacitor_SMD:C_0402_1005Metric, F.Cu at (200.1, 123.0)
- added D17: Blue, AT-LED:LED0603, F.Cu at (-36.6, 183.8)
- added D18: Red, AT-LED:LED0603, F.Cu at (205.3, 113.0)
- added H1: M3, MountingHole:MountingHole_3.2mm_M3_Pad, F.Cu at (172.0, 113.0)
- added H2: M3, MountingHole:MountingHole_3.2mm_M3_Pad, F.Cu at (228.0, 201.0)
- added H3: M3, MountingHole:MountingHole_3.2mm_M3_Pad, F.Cu at (172.0, 186.0)
- added H4: M3, MountingHole:MountingHole_3.2mm_M3_Pad, F.Cu at (228.0, 100.0)
- added J14: Conn_01x08, Connector_JST:JST_SH_SM08B-SRSS-TB_1x08-1MP_P1.00mm_Horizontal, B.Cu at (171.0, 198.5)
- added J15: Conn_01x08, Connector_JST:JST_SH_SM08B-SRSS-TB_1x08-1MP_P1.00mm_Horizontal, B.Cu at (171.0, 102.0)
- added J16: Conn_01x04_Pin, Connector_PinHeader_2.54mm:PinHeader_1x04_P2.54mm_Vertical, F.Cu at (-134.0, 149.4)
- added L8: 650 @100MHz, Resistor_SMD:R_0603_1608Metric, F.Cu at (-36.6, 186.4)
- added P1: USB_C_Plug_USB2.0, Connector_USB:USB_C_Receptacle_Molex_105450-0101, F.Cu at (201.0, 200.0)
- added R78: 10k, Resistor_SMD:R_0402_1005Metric, F.Cu at (-21.5, 165.1)
- added R79: 2.1k, Resistor_SMD:R_0402_1005Metric, F.Cu at (-16.6, 165.1)
- added R80: 2.1k, Resistor_SMD:R_0402_1005Metric, F.Cu at (-16.6, 167.1)
- added R81: 2.1k, Resistor_SMD:R_0402_1005Metric, F.Cu at (-16.6, 169.1)
- added R82: 2.1k, Resistor_SMD:R_0402_1005Metric, F.Cu at (-16.6, 171.0)
- added R83: 10k, Resistor_SMD:R_0402_1005Metric, F.Cu at (-21.5, 167.1)
- added R84: 330, Resistor_SMD:R_0402_1005Metric, F.Cu at (-21.5, 169.1)
- added R85: 330, Resistor_SMD:R_0402_1005Metric, F.Cu at (-21.5, 171.0)
- added R86: 330, Resistor_SMD:R_0402_1005Metric, F.Cu at (-21.5, 173.0)
- added R87: 330, Resistor_SMD:R_0402_1005Metric, F.Cu at (-21.5, 175.0)
- added R88: 330, Resistor_SMD:R_0402_1005Metric, F.Cu at (-21.5, 177.0)
- added R89: 5.1k, Resistor_SMD:R_0402_1005Metric, F.Cu at (-21.5, 179.0)
- added R90: 2.2k, Resistor_SMD:R_0402_1005Metric, F.Cu at (205.3, 110.2)
- added RV1: ACFG1, Potentiometer_SMD:Potentiometer_Bourns_3269X_Horizontal, B.Cu at (172.0, 161.0)
- added RV2: ACFG2, Potentiometer_SMD:Potentiometer_Bourns_3269X_Horizontal, B.Cu at (172.0, 139.0)
- added U14: STM32F407VETx, Package_QFP:LQFP-100_14x14mm_P0.5mm, F.Cu at (200.0, 150.0)
- C54: value 1u 50V -> 100n 50V
- J11: value Conn_01x06 -> Conn_01x08; footprint Connector_JST:JST_SH_SM06B-SRSS-TB_1x06-1MP_P1.00mm_Horizontal -> Connector_JST:JST_SH_SM08B-SRSS-TB_1x08-1MP_P1.00mm_Horizontal; moved to B.Cu
- R15: footprint Resistor_SMD:R_0402_1005Metric -> Resistor_SMD:R_0603_1608Metric
- SW4: moved to B.Cu
- U12: footprint Package_CSP:WLCSP-8_1.58x1.63x0.35mm_Layout3x5_P0.35x0.4mm_Ball0.25mm_Pad0.25mm_NSMD -> Package_SO:SOIC-8_3.9x4.9mm_P1.27mm
- moved D11 373.9 mm to (248.8, 96.0)
- moved J3 326.5 mm to (241.0, 201.0)
- moved Q1 296.4 mm to (-90.3, 170.6)
- moved R5 296.4 mm to (-93.3, 173.3)
- moved U10 290.1 mm to (247.2, 153.6), turned to -90 degrees
- moved U5 287.5 mm to (190.0, 195.0)
- moved C34 286.6 mm to (248.9, 160.0), turned to -90 degrees
- moved C35 284.4 mm to (246.4, 159.2), turned to -90 degrees
- moved J10 275.8 mm to (171.0, 132.0), turned to -90 degrees
- moved U6 275.5 mm to (180.0, 195.0)
- moved J13 256.1 mm to (175.6, 176.0), turned to 90 degrees
- moved R32 250.8 mm to (203.9, 120.1), turned to -90 degrees
- moved J8 250.6 mm to (171.0, 196.0), turned to -90 degrees
- moved L5 249.2 mm to (201.4, 107.2), turned to 90 degrees
- moved C9 249.1 mm to (203.9, 123.0), turned to -90 degrees
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Connections:
- net /digital/DIP0 renamed Net-(R40-Pad2)
- net /digital/DIP1 renamed Net-(R39-Pad2)
- net /digital/DIP2 renamed Net-(R38-Pad2)
- net /digital/DIP3 renamed Net-(R37-Pad2)
- C23 pad 1: /digital/USR_BTN -> Net-(C23-Pad1)
- C53 pad 1: Net-(U4-VDDA) -> +3V3
- C54 pad 1: Net-(U4-VDDA) -> +3V3
- C55 pad 2: Net-(U4-VCAP1) -> +3V3
- D16 pad 3: /digital/V_{sense}_12v0 -> /digital/USB_OTG_FS_DM
- D16 pad 4: /digital/V_{sense}_6v2 -> /digital/USB_OTG_FS_DP
- J11 pad 1: +5V -> +3V3
- J11 pad 2: +3V3 -> /Breakbeam/BB_CENTER.AGPIO
- J11 pad 3: /Breakbeam/BB_BUS.SDA -> GND
- J11 pad 4: /Breakbeam/BB_BUS.SCL -> /Breakbeam/BB_CENTER.SDA
- J11 pad 5: /Breakbeam/BB_BUS.RST -> /Breakbeam/BB_CENTER.SCL
- J11 pad 6: GND -> /Breakbeam/BB_CENTER.RST
- J3 pad 10: /digital/SERVO_LIM2 -> /digital/AUX_GPIO2
- J3 pad 5: /digital/SERVO_SS -> /digital/AUX_NSS
- J3 pad 6: /digital/FLASH_SCK -> /digital/AUX_SCK
- J3 pad 7: /digital/FLASH_MISO -> /digital/AUX_MISO
- J3 pad 8: /digital/FLASH_MOSI -> /digital/AUX_MOSI
- J3 pad 9: /digital/SERVO_LIM1 -> /digital/AUX_GPIO1
- J8 pad 2: /Breakbeam/BB_BUS.BB_{TX} -> /Breakbeam/BB_LEFT.AGPIO
- J9 pad 2: /Breakbeam/BB_BUS.BB_{RX} -> /Breakbeam/BB_RIGHT.AGPIO
- R34 pad 1: /digital/USR_BTN -> Net-(C23-Pad1)
- R35 pad 1: /digital/BB_LED_BLUE -> /digital/BB_LED2_BLUE
- R74 pad 2: /Breakbeam/BB_BUS.SDA -> /Breakbeam/BB_CENTER.SDA
- R75 pad 2: /Breakbeam/BB_BUS.SCL -> /Breakbeam/BB_CENTER.SCL
- SW3 pad 1: /digital/USR_BTN -> Net-(C23-Pad1)
- U3 pad 10: (no net) -> GND
- U3 pad 18: (no net) -> GND
- U3 pad 23: (no net) -> /digital/PGOOD
- U3 pad 27: (no net) -> GND
Routing:
- net /digital/AUX_GPIO2: track 0.00 -> 76.5 mm
- net /digital/AUX_GPIO1: track 0.00 -> 75.5 mm
- net /digital/AUX_MOSI: track 0.00 -> 73.4 mm
- net /digital/AUX_MISO: track 0.00 -> 72.5 mm
- net /digital/AUX_SCK: track 0.00 -> 71.5 mm
- net /digital/AUX_NSS: track 0.00 -> 70.5 mm
- net /Power Protection/PGOOD_{VBATT}: track 0.00 -> 11.7 mm, vias 0 -> 2
- net /digital/PGOOD: track 0.00 -> 5.94 mm
- net /Power Protection/V_{BATT}_FUSED: track 31.9 -> 26.9 mm
- net Net-(U3D-RUN/SS3): track 0.00 -> 4.75 mm
- net /isol/BOOT_UART_RST_ISOL: track 4.69 -> 9.34 mm
- net /isol/BOOT_UART_BOOT0_ISOL: track 4.58 -> 9.22 mm
- net Net-(U3C-RUN/SS2): track 0.00 -> 3.37 mm
- net /digital/PWR_KILL: track 5.48 -> 2.15 mm
- net Net-(U3A-RT/SYNC): track 0.00 -> 3.23 mm
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- added copper zone on F.Cu, net Net-(C11-Pad1)
- added copper zone on F.Cu, net Net-(C12-Pad1)
- added copper zone on F.Cu, net Net-(C13-Pad1)
- added copper zone on F.Cu, net Net-(C14-Pad1)
- added copper zone on F.Cu, net Net-(D4-A)
- added copper zone on F.Cu, net Net-(D4-K)
- added copper zone on F.Cu, net Net-(D5-A)
- added copper zone on F.Cu, net Net-(D5-K)
- added copper zone on F.Cu, net Net-(D6-A)
- added copper zone on F.Cu, net Net-(D6-K)
- added copper zone on F.Cu, net Net-(D7-A)
- added copper zone on F.Cu, net Net-(D7-K)
- added copper zone on F.Cu, net Net-(U3A-SKY)
- added copper zone on F.Cu, net Net-(U3A-SW5)

Commit message: kicker layout work
Parts:
- D11, D12: footprint AT-LED:LED0603 -> AT-LED:APA1606
- J12, U13: moved to B.Cu
- SW4: footprint Button_Switch_SMD:SW_DIP_SPSTx04_Slide_Omron_A6S-410x_W8.9mm_P2.54mm -> at-switches:CHP-041TB
- moved D12 400.0 mm to (255.0, 203.5), turned to 180 degrees
- moved R45 398.6 mm to (255.0, 190.8), turned to -90 degrees
- moved R44 398.2 mm to (255.0, 187.0), turned to -90 degrees
- moved R42 384.3 mm to (254.2, 113.5), turned to 90 degrees
- moved R43 383.7 mm to (254.2, 109.8), turned to 90 degrees
- moved U13 315.8 mm to (228.8, 191.2), turned to 180 degrees
- moved J12 312.5 mm to (237.0, 201.0), turned to 180 degrees
- moved J2 294.6 mm to (214.0, 138.4), turned to 90 degrees
- moved R50 273.4 mm to (253.2, 154.6)
- moved R51 273.4 mm to (253.2, 156.5)
- moved R52 273.4 mm to (253.2, 158.5)
- moved R53 273.4 mm to (253.2, 160.5)
- moved R54 273.4 mm to (253.2, 162.5)
- moved R55 273.4 mm to (253.2, 164.5)
- moved R3 271.5 mm to (238.8, 119.5), turned to 135 degrees
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Routing:
- net +5V: track 0.00 -> 135.7 mm, vias 0 -> 2
- net +6V: track 0.00 -> 94.7 mm, vias 0 -> 2
- net /digital/MCU_BOOT_UART.TX: track 0.00 -> 43.2 mm, vias 0 -> 2
- net +3V3: track 5.06 -> 48.3 mm, vias 0 -> 8
- net /digital/MCU_BOOT_UART.RX: track 0.00 -> 42.3 mm, vias 0 -> 2
- net Net-(U3B-FB1): track 0.00 -> 33.4 mm, vias 0 -> 2
- net Net-(U3D-FB3): track 0.00 -> 32.4 mm, vias 0 -> 2
- net Net-(U3E-FB4): track 0.00 -> 21.5 mm, vias 0 -> 2
- net Net-(U3C-FB2): track 0.00 -> 18.5 mm, vias 0 -> 2
- net Net-(D11-A): track 0.00 -> 13.1 mm
- net Net-(D12-A): track 0.00 -> 12.2 mm
- net /digital/USB_OTG_FS_DM: track 0.00 -> 10.6 mm
- net /digital/USB_OTG_FS_DP: track 0.00 -> 10.4 mm
- net +BATT: track 29.4 -> 37.7 mm, vias 48 -> 57
- net /digital/SWDIO: track 0.00 -> 8.26 mm
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- added copper zone on B.Cu, net +3V3
