File: robot/control/v2.0.0/control/control.kicad_pcb (KiCad board)
At the start: 6 copper layers, 140 x 105 mm, 518 parts, among them J1 EC3-M, J10 SM06B-SRSS-TB, J11 S08B-PASK-2, J12 SM06B-SRSS-TB, J13 S08B-PASK-2, J14 SM06B-SRSS-TB, J15 BM10B-SRSS-TB, J16 BM11B-SRSS-TB, J17 XT30PW-F, J18 SM10B-SRSS-TB, J19 BM09B-SRSS-TB, J2 10033527-N3112MLF, J20 BM09B-SRSS-TB, J21 B04B-ZESK-1D, J22 B04B-ZESK-1D, J3 ARM_SWD, J4 MEM2067-02-180-00-A, J5 S08B-PASK-2, J6 SM06B-SRSS-TB, J7 S08B-PASK-2, J8 SM06B-SRSS-TB, J9 S08B-PASK-2, Q1 SQJA80EP-T1_GE3, Q10 STL90N10F7, Q11 STL90N10F7, Q12 STL90N10F7, Q13 STL90N10F7, Q14 STL90N10F7, Q15 STL90N10F7, Q16 STL90N10F7, Q17 STL90N10F7, Q18 STL90N10F7, Q19 STL90N10F7, Q2 SQJA80EP-T1_GE3, Q20 STL90N10F7, Q21 STL90N10F7, Q22 STL90N10F7, Q23 STL90N10F7, Q24 STL90N10F7, Q25 STL90N10F7, Q26 STL90N10F7, Q27 STL90N10F7, Q28 STL90N10F7, Q29 STL90N10F7, Q3 BSS138K, Q30 STL90N10F7, Q31 STL90N10F7, Q32 STL90N10F7, Q33 STL90N10F7, Q34 STL90N10F7, Q35 STL90N10F7, Q36 STL90N10F7, Q37 STL90N10F7, Q4 BSS138K, Q5 BSS138K, Q6 BSS138K, Q7 BSS138K, Q8 STL90N10F7, Q9 STL90N10F7, SW1 HDR_2P, SW2 CPG151101D91, SW3 221ADC16, SW4 TS02-66-73-BK-160-SCR-D, SW5 TS02-66-73-BK-160-SCR-D, SW6 219-8MST, SW7 TS02-66-73-BK-160-SCR-D, U1 LTC4367, U10 STSPIN32F0B, U11 STSPIN32F0B, U12 STSPIN32F0B, U13 STSPIN32F0B, U14 STSPIN32F0B, U2 LTC2955-1, U3 TPS54260DGQ, U4 TPS54260DGQ, U5 TPS54561DPR, U6 TPS54561DPR, U7 SK9822, U8 SK9822, U9 STM32H723ZGT6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

Commit message: WIP
Parts:
- removed the D36 at (232.0, 157.0)
- removed the D42 at (256.8, 43.6)
- added D46: BAS16VY, Package_TO_SOT_SMD:SOT-363_SC-70-6, F.Cu at (47.7, 51.2)
- added D47: BAS16VY, Package_TO_SOT_SMD:SOT-363_SC-70-6, F.Cu at (55.0, 52.0)
- moved U2 316.6 mm to (159.0, 47.5)
- moved R13 307.8 mm to (159.0, 53.5)
- moved R12 306.3 mm to (159.0, 52.0)
- moved J1 277.4 mm to (140.5, 59.2), turned to 180 degrees
- moved D37 270.5 mm to (228.5, 158.5)
- moved J15 253.1 mm to (121.5, 134.0), turned to -90 degrees
- moved BZ1 248.2 mm to (124.0, 148.5), turned to 90 degrees
- moved J16 241.6 mm to (109.8, 103.0)
- moved D8 239.0 mm to (129.0, 148.5), turned to 90 degrees
- moved D12 238.8 mm to (126.0, 154.5), turned to 180 degrees
- moved R36 232.7 mm to (122.0, 143.0)
- moved R46 231.9 mm to (122.5, 158.0)
- moved D9 230.3 mm to (126.0, 152.8), turned to 180 degrees
- moved C33 230.1 mm to (98.0, 105.2)
- moved R35 229.1 mm to (122.0, 144.0)
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- renumbered D37 to D36, D38 to D37, D39 to D38, D40 to D39, D41 to D40, D43 to D41, D44 to D42, D45 to D43, D46 to D44, D47 to D45
Connections:
- D36 pad 2: Net-(D37B-A) (its old number) -> Net-(D36B-A)
- D36 pad 5: Net-(D37B-K) (its old number) -> Net-(D36B-K)
- D37 pad 3: Net-(D38C-A) -> Net-(D37C-A)
- D37 pad 4: Net-(D38C-K) -> Net-(D37C-K)
- D41 pad 2: Net-(D43B-A) -> Net-(D41B-A)
- D41 pad 3: Net-(D43C-A) -> Net-(D41C-A)
- D41 pad 4: Net-(D43C-K) -> Net-(D41C-K)
- D41 pad 5: Net-(D43B-K) -> Net-(D41B-K)
- D42 pad 2: Net-(D44B-A) -> Net-(D42B-A)
- D42 pad 3: Net-(D44C-A) -> Net-(D42C-A)
- D42 pad 4: Net-(D44C-K) -> Net-(D42C-K)
- D42 pad 5: Net-(D44B-K) -> Net-(D42B-K)
- R166 pad 1: Net-(D36C-A) (its old number) -> Net-(D37C-A)
- R167 pad 1: Net-(D36C-K) (its old number) -> Net-(D37C-K)
- R192 pad 1: Net-(D42B-A) -> Net-(D41B-A)
- R193 pad 1: Net-(D42B-K) -> Net-(D41B-K)
- R194 pad 1: Net-(D38C-K) -> Net-(D41C-K)
- R195 pad 1: Net-(D38C-A) -> Net-(D41C-A)
- R202 pad 1: Net-(D37B-K) (its old number) -> Net-(D42B-K)
- R203 pad 1: Net-(D37B-A) (its old number) -> Net-(D42B-A)
- R222 pad 1: Net-(D43B-A) -> Net-(D46B-A)
- R223 pad 1: Net-(D43B-K) -> Net-(D46B-K)
- R224 pad 1: Net-(D43C-K) -> Net-(D46C-K)
- R225 pad 1: Net-(D43C-A) -> Net-(D46C-A)
- R226 pad 1: Net-(D44C-A) -> Net-(D47C-A)
- R227 pad 1: Net-(D44C-K) -> Net-(D47C-K)
- R232 pad 1: Net-(D44B-K) -> Net-(D47B-K)
- R233 pad 1: Net-(D44B-A) -> Net-(D47B-A)
- U12 pad 29: Net-(D36C-K) (its old number) -> Net-(D37C-K)
- U13 pad 28: Net-(D37B-K) (its old number) -> Net-(D42B-K)
- U13 pad 33: Net-(D42B-K) -> Net-(D41B-K)
- U13 pad 36: Net-(D38C-K) -> Net-(D41C-K)
- U14 pad 28: Net-(D44B-K) -> Net-(D47B-K)
- U14 pad 29: Net-(D44C-K) -> Net-(D47C-K)
- U14 pad 33: Net-(D43B-K) -> Net-(D46B-K)
- U14 pad 36: Net-(D43C-K) -> Net-(D46C-K)
- U9 pad 114: /Indicators/ROBOTID_{DISP}.FR -> /Indicators/ROBOTID_{DISP}.FL
- U9 pad 115: /Indicators/ROBOTID_{DISP}.FL -> /Indicators/ROBOTID_{DISP}.BL
- U9 pad 117: /Indicators/ROBOTID_{DISP}.BL -> /Indicators/ROBOTID_{DISP}.BR
- U9 pad 118: /Indicators/ROBOTID_{DISP}.BR -> /Indicators/ROBOTID_{DISP}.FR
Routing:
- net /MCU/~{RST}: track 0.00 -> 85.1 mm, vias 0 -> 2
- net /KICKER.PWRON: track 0.00 -> 63.2 mm
- net /KICKER.TX: track 0.00 -> 58.8 mm
- net /KICKER.RX: track 0.00 -> 58.1 mm
- net /KICKER.BOOT0: track 0.00 -> 56.6 mm
- net /KICKER.~{RST}: track 0.00 -> 55.9 mm
- net /USB_OTG.ID: track 4.19 -> 57.8 mm, vias 0 -> 2
- net /Motors/MotorFL/HALL_{2}: track 2.54 -> 50.8 mm, vias 0 -> 1
- net /Indicators/LED.3: track 0.00 -> 48.0 mm
- net /Indicators/DOTSTAR.CLK: track 0.00 -> 47.1 mm, vias 0 -> 2
- net /Indicators/LED.2: track 0.00 -> 46.7 mm
- net /Indicators/DOTSTAR.DAT: track 0.00 -> 46.0 mm, vias 0 -> 2
- net /Indicators/LED.1: track 0.00 -> 45.4 mm
- net /Motors/MotorFL/HALL_{1}: track 2.40 -> 47.1 mm, vias 0 -> 1
- net /MCU/IsBlueTeam: track 0.00 -> 44.2 mm, vias 0 -> 2
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- added copper zone on F.Cu, net (none)
- added copper zone on F.Cu, net /Motors/MotorBL/MOTOR_{U}
- added copper zone on In1.Cu, net /Motors/MotorBL/MOTOR_{U}
- added copper zone on In4.Cu, net /Motors/MotorBL/MOTOR_{U}
- added copper zone on F.Cu, net /Motors/MotorBL/MOTOR_{V}
- added copper zone on In1.Cu, net /Motors/MotorBL/MOTOR_{V}
- added copper zone on In4.Cu, net /Motors/MotorBL/MOTOR_{V}
- added copper zone on F.Cu, net /Motors/MotorBL/MOTOR_{W}
- added copper zone on In1.Cu, net /Motors/MotorBL/MOTOR_{W}
- added copper zone on In4.Cu, net /Motors/MotorBL/MOTOR_{W}
Other:
- board size 140 x 105 mm -> 148 x 121 mm

Commit message: WIP
Parts:
- added C119: 0.1uF 63V, Capacitor_SMD:C_0402_1005Metric, F.Cu at (106.5, 108.0)
- added C120: 0.1uF 63V, Capacitor_SMD:C_0402_1005Metric, F.Cu at (104.5, 108.0)
- added R237: 4.7k, Resistor_SMD:R_0402_1005Metric, F.Cu at (110.0, 113.2)
- added R238: 4.7k, Resistor_SMD:R_0402_1005Metric, F.Cu at (107.0, 113.2)
- added R239: 100, Resistor_SMD:R_0402_1005Metric, F.Cu at (109.0, 113.2)
- added R240: 100, Resistor_SMD:R_0402_1005Metric, F.Cu at (108.0, 113.2)
- added U15: BMI323, AT-IMU:BMI323, F.Cu at (105.0, 105.0)
- Q26, Q27, Q28, Q29, Q30, Q31, R204: moved to B.Cu
- moved L4 188.8 mm to (125.2, 97.8), turned to -90 degrees
- moved D6 188.3 mm to (121.2, 91.5), turned to 180 degrees
- moved D17 180.7 mm to (166.0, 55.0), turned to 180 degrees
- moved C29 178.9 mm to (123.5, 104.0), turned to 180 degrees
- moved JP4 178.5 mm to (130.5, 104.0)
- moved F9 173.1 mm to (127.5, 104.0)
- moved C21 171.4 mm to (120.5, 99.2), turned to -90 degrees
- moved C19 171.0 mm to (115.5, 91.5)
- moved C27 170.6 mm to (118.0, 89.2)
- moved C23 169.4 mm to (118.5, 99.2), turned to 90 degrees
- moved U6 168.6 mm to (118.0, 95.8), turned to 90 degrees
- moved R26 167.5 mm to (119.5, 99.2), turned to -90 degrees
- moved C25 164.8 mm to (114.0, 99.2), turned to -90 degrees
- moved R30 163.3 mm to (118.0, 88.2)
- moved R28 163.0 mm to (115.0, 99.2), turned to -90 degrees
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- renumbered C119 to C121, C120 to C122, R237 to R241
Connections:
- C107 pad 1: /Motors/MotorDRB/V_{MOTOR} -> +V_{BATT(PROTECTED)}
- C59 pad 1: /Motors/MotorFL/V_{MOTOR} -> +V_{BATT(PROTECTED)}
- C71 pad 1: /Motors/MotorBL/V_{MOTOR} -> +V_{BATT(PROTECTED)}
- C83 pad 1: /Motors/MotorBR/V_{MOTOR} -> +V_{BATT(PROTECTED)}
- C95 pad 1: /Motors/MotorFR/V_{MOTOR} -> +V_{BATT(PROTECTED)}
- U9 pad 40: unconnected-(U9B-PA4-Pad40) -> /IMU.~{SS}0
Routing:
- net Net-(R70-Pad1): track 53.9 -> 4.35 mm, vias 2 -> 1
- net /Indicators/LED.3: track 48.0 -> 5.28 mm
- net /Indicators/LED.2: track 46.7 -> 5.49 mm
- net /Indicators/LED.1: track 45.4 -> 5.70 mm
- net /MCU/SDMMC.D1: track 18.9 -> 58.3 mm
- net /MCU/SDMMC.D0: track 18.8 -> 58.1 mm
- net /Indicators/LED.0: track 44.1 -> 5.91 mm
- net /MCU/BOOT0: track 3.68 -> 35.5 mm, vias 0 -> 2
- net Net-(R73-Pad2): track 29.2 -> 0.00 mm, vias 2 -> 1
- net Net-(R74-Pad2): track 28.6 -> 0.00 mm, vias 2 -> 1
- net Net-(R72-Pad2): track 28.4 -> 0.00 mm, vias 2 -> 1
- net Net-(R75-Pad2): track 28.0 -> 0.00 mm, vias 2 -> 1
- net Net-(R76-Pad2): track 27.6 -> 0.00 mm, vias 2 -> 1
- net Net-(R77-Pad2): track 27.0 -> 0.00 mm, vias 2 -> 1
- net Net-(R78-Pad2): track 26.2 -> 0.00 mm, vias 2 -> 1
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- added copper zone on B.Cu, net /Motors/MotorFR/I_{SENSE(RAW)}
- added copper zone on F.Cu, net Net-(D6-K)
- removed copper zone on F.Cu, net (none)
Other:
- board text added: "+X"
- board text added: "+Y"
