File: robot/control/v2.0.0/control/control.kicad_sch (KiCad schematic)
At the start: 14 parts, among them J1 EC3-M, J9 10033527-N3112MLF

Commit message: WIP
Parts:
- J1: footprint AT-Connectors:XT60-M_TH_WireMount -> AT-Connectors:EC3-M_TH_WireMount
Changed lines of the file:
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@@
     (comment 1 "W. Stuckey & R. Osawa")
   )
+  (bus_alias "RADIO" (members "RADIO.~{RST}" "RADIO.BOOT0" "RADIO.TX" "RADIO.RX" "RADIO.CTS" "RADIO.RTS" "RADIO.~{DET}"))
+  (bus_alias "EXTLOGIC" (members "EXTLOGIC.TX" "EXTLOGIC.RX" "EXTLOGIC.CK" "EXTLOGIC.NSS" "EXTLOGIC.~{DET}"))
   (bus_alias "SDMMC" (members "SDMMC.CMD" "SDMMC.D0" "SDMMC.D1" "SDMMC.D2" "SDMMC.D3" "SDMMC.CK"))
+  (bus_alias "FLOW" (members "FLOW.TX" "FLOW.RX" "FLOW.BOOT0" "FLOW.~{RST}" "FLOW.~{DET}"))
   (bus_alias "KICKER" (members "KICKER.~{DET}" "KICKER.PWRON" "KICKER.TX" "KICKER.RX" "KICKER.BOOT0" "KICKER.~{RST}"))
-  (bus_alias "FLOW" (members "FLOW.TX" "FLOW.RX" "FLOW.BOOT0" "FLOW.~{RST}" "FLOW.~{DET}"))
-  (bus_alias "EXTLOGIC" (members "EXTLOGIC.TX" "EXTLOGIC.RX" "EXTLOGIC.CK" "EXTLOGIC.NSS" "EXTLOGIC.~{DET}"))
-  (bus_alias "RADIO" (members "RADIO.~{RST}" "RADIO.BOOT0" "RADIO.TX" "RADIO.RX" "RADIO.CTS" "RADIO.RTS" "RADIO.~{DET}"))
   (bus_alias "IMU" (members "IMU.~{SS}1" "IMU.~{SS}2" "IMU.~{SS}3" "IMU.MOSI" "IMU.MISO" "IMU.SCK" "IMU.INT1" "IMU.INT2" "IMU.~{DET}" "IMU.~{SS}0"))
   (junction (at 40.64 24.13) (diameter 0) (color 0 0 0 0)
@@
       (effects (font (size 1.27 1.27)))
     )
-    (property "Footprint" "AT-Connectors:XT60-M_TH_WireMount" (at 33.02 26.67 0)
-      (effects (font (size 1.27 1.27)) hide)
-    )
+    (property "Footprint" "AT-Connectors:EC3-M_TH_WireMount" (at 33.02 26.67 0)
+      (effects (font (size 1.27 1.27)) hide)
+    )

Commit message: WIP
Parts:
- added R57: 130k, Resistor_SMD:R_0402_1005Metric, symbol Device:R_Small_US
- added R57: 11k, Resistor_SMD:R_0402_1005Metric, symbol Device:R_Small_US
Connections:
- net +V_{BATT(PROTECTED)}: now also R57.1
- net GND: now also R57.2
- new net MCU/+V_{BATT(REDUCED)}: R57.1, R57.2
Other:
- sheet MCU ports: added +V_{BATT(REDUCED)}; removed none
- moved on the sheet: TP2, TP3, TP4, TP5

Commit message: WIP
Parts:
- added Q3: SI2310-TP, Package_TO_SOT_SMD:SOT-23, symbol Device:Q_NMOS_GSD
- added R10: 10, Resistor_SMD:R_0402_1005Metric, symbol Device:R_Small_US
- added R57: 1k, Resistor_SMD:R_0402_1005Metric, symbol Device:R_Small_US
- added U1: ITS4140N, Package_TO_SOT_SMD:SOT-223, symbol AT-PowerIC:ITS4140N
- renumbered J1 to J2
Connections:
- net +3.3V: now also R10.2
- net +V_{BATT(PROTECTED)}: now also U1.2 (V_{bb}), U1.4 (V_{bb}); no longer R57.1
- net GND: now also Q3.2 (S), R57.2
- new net: Q3.1 (G), R10.1, R57.1
- new net: R57.1, U1.3 (OUT)
- new net: Q3.3 (D), U1.1 (IN)
Other:
- moved on the sheet: J9, R57, TP2, TP3, TP4, TP5

Commit message: Control v2.0 pre minor mods for manufacturing
Parts:
- R57: value 1k -> 4.7k
Changed lines of the file:
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@@
     (comment 1 "W. Stuckey & R. Osawa")
   )
+  (bus_alias "FLOW" (members "FLOW.TX" "FLOW.RX" "FLOW.BOOT0" "FLOW.~{RST}" "FLOW.~{DET}"))
+  (bus_alias "RADIO" (members "RADIO.~{RST}" "RADIO.BOOT0" "RADIO.TX" "RADIO.RX" "RADIO.CTS" "RADIO.RTS" "RADIO.~{DET}"))
   (bus_alias "SDMMC" (members "SDMMC.CMD" "SDMMC.D0" "SDMMC.D1" "SDMMC.D2" "SDMMC.D3" "SDMMC.CK"))
+  (bus_alias "EXTLOGIC" (members "EXTLOGIC.TX" "EXTLOGIC.RX" "EXTLOGIC.CK" "EXTLOGIC.NSS" "EXTLOGIC.~{DET}"))
   (bus_alias "KICKER" (members "KICKER.~{DET}" "KICKER.PWRON" "KICKER.TX" "KICKER.RX" "KICKER.BOOT0" "KICKER.~{RST}"))
   (bus_alias "IMU" (members "IMU.~{SS}1" "IMU.~{SS}2" "IMU.~{SS}3" "IMU.MOSI" "IMU.MISO" "IMU.SCK" "IMU.INT1" "IMU.INT2" "IMU.~{DET}" "IMU.~{SS}0"))
-  (bus_alias "EXTLOGIC" (members "EXTLOGIC.TX" "EXTLOGIC.RX" "EXTLOGIC.CK" "EXTLOGIC.NSS" "EXTLOGIC.~{DET}"))
-  (bus_alias "RADIO" (members "RADIO.~{RST}" "RADIO.BOOT0" "RADIO.TX" "RADIO.RX" "RADIO.CTS" "RADIO.RTS" "RADIO.~{DET}"))
-  (bus_alias "FLOW" (members "FLOW.TX" "FLOW.RX" "FLOW.BOOT0" "FLOW.~{RST}" "FLOW.~{DET}"))
   (junction (at 40.64 24.13) (diameter 0) (color 0 0 0 0)
   )
@@
       (effects (font (size 1.27 1.27)) (justify left))
     )
-    (property "Value" "1k" (at 80.01 160.655 0)
+    (property "Value" "4.7k" (at 80.01 160.655 0)
       (effects (font (size 1.27 1.27)) (justify left))
     )

Commit message: Control v2.0 for DFM review
Parts:
- D1: value 824521261 -> SMBJ26CA
- J9: value 10033527-N3112MLF -> 10033526-N3212LF; footprint AT-Connectors:10033527-N3112MLF -> AT-Connectors:10033526-N3212LF
Changed lines of the file:
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@@
     (comment 1 "W. Stuckey & R. Osawa")
   )
+  (bus_alias "IMU" (members "IMU.~{SS}1" "IMU.~{SS}2" "IMU.~{SS}3" "IMU.MOSI" "IMU.MISO" "IMU.SCK" "IMU.INT1" "IMU.INT2" "IMU.~{DET}" "IMU.~{SS}0"))
+  (bus_alias "RADIO" (members "RADIO.~{RST}" "RADIO.BOOT0" "RADIO.TX" "RADIO.RX" "RADIO.CTS" "RADIO.RTS" "RADIO.~{DET}"))
   (bus_alias "FLOW" (members "FLOW.TX" "FLOW.RX" "FLOW.BOOT0" "FLOW.~{RST}" "FLOW.~{DET}"))
-  (bus_alias "RADIO" (members "RADIO.~{RST}" "RADIO.BOOT0" "RADIO.TX" "RADIO.RX" "RADIO.CTS" "RADIO.RTS" "RADIO.~{DET}"))
+  (bus_alias "KICKER" (members "KICKER.~{DET}" "KICKER.PWRON" "KICKER.TX" "KICKER.RX" "KICKER.BOOT0" "KICKER.~{RST}"))
   (bus_alias "SDMMC" (members "SDMMC.CMD" "SDMMC.D0" "SDMMC.D1" "SDMMC.D2" "SDMMC.D3" "SDMMC.CK"))
   (bus_alias "EXTLOGIC" (members "EXTLOGIC.TX" "EXTLOGIC.RX" "EXTLOGIC.CK" "EXTLOGIC.NSS" "EXTLOGIC.~{DET}"))
-  (bus_alias "KICKER" (members "KICKER.~{DET}" "KICKER.PWRON" "KICKER.TX" "KICKER.RX" "KICKER.BOOT0" "KICKER.~{RST}"))
-  (bus_alias "IMU" (members "IMU.~{SS}1" "IMU.~{SS}2" "IMU.~{SS}3" "IMU.MOSI" "IMU.MISO" "IMU.SCK" "IMU.INT1" "IMU.INT2" "IMU.~{DET}" "IMU.~{SS}0"))
   (junction (at 40.64 24.13) (diameter 0) (color 0 0 0 0)
   )
@@
       (effects (font (size 1.27 1.27)))
     )
-    (property "Value" "10033527-N3112MLF" (at 27.94 144.78 0)
-      (effects (font (size 1.27 1.27)))
-    )
-    (property "Footprint" "AT-Connectors:10033527-N3112MLF" (at 31.75 156.21 0)
+    (property "Value" "10033526-N3212LF" (at 27.94 144.78 0)
+      (effects (font (size 1.27 1.27)))
+    )
+    (property "Footprint" "AT-Connectors:10033526-N3212LF" (at 31.75 156.21 0)
       (effects (font (size 1.27 1.27)) hide)
     )
@@
       (effects (font (size 1.27 1.27)) (justify right))
     )
-    (property "Value" "824521261" (at 71.12 30.48 90)
+    (property "Value" "SMBJ26CA" (at 71.12 30.48 90)
       (effects (font (size 1.27 1.27)) (justify right))
     )
