File: robot/control/v2.0.0/control/air_dribbler.kicad_sch (KiCad schematic)
At the start: 4 parts, among them J7 B04B-ZESK-1D

Commit message: WIP
Parts:
- J7: value B04B-ZESK-1D -> SM04B-ZESS-TB; footprint Connector_JST:JST_ZE_B04B-ZESK-1D_1x04_P1.50mm_Vertical -> Connector_JST:JST_ZE_BM03B-ZESS-TBT_1x03-1MP_P1.50mm_Vertical; symbol Connector_Generic:Conn_01x04 -> Connector_Generic_MountingPin:Conn_01x03_MountingPin
Connections:
- net AIRDRIBBLER.PWM1: now also J7.3 (Pin_3); no longer J7.4 (Pin_4)
- net AIRDRIBBLER.PWM2: now also J7.3 (Pin_3); no longer J7.4 (Pin_4)
- net GND: now also J7.MP (MountPin), J7.MP (MountPin)
- no-connect marks 2 -> 0
Other:
- note added: "3 Blue X Green 2 Yellow 1 Black"
- note removed: "4 Blue 3 Green 2 Yellow 1 Black"
- moved on the sheet: C30

Commit message: Fix connector part number
Parts:
- J7: value SM04B-ZESS-TB -> BM03B-ZESS-TBT
Changed lines of the file:
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@@
       (effects (font (size 1.27 1.27)))
     )
-    (property "Value" "SM04B-ZESS-TB" (at 69.85 34.29 90)
+    (property "Value" "BM03B-ZESS-TBT" (at 69.85 34.29 90)
       (effects (font (size 1.27 1.27)))
     )
@@
       (effects (font (size 1.27 1.27)))
     )
-    (property "Value" "SM04B-ZESS-TB" (at 69.85 63.5 90)
-      (effects (font (size 1.27 1.27)))
-    )
+    (property "Value" "BM03B-ZESS-TBT" (at 69.85 63.5 90)
+      (effects (font (size 1.27 1.27)))
+    )

Commit message: Update title block
Other:
- company: (none) -> The A-Team (RC SSL)
Changed lines of the file:
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@@
 (kicad_sch (version 20230121) (generator eeschema)
   (paper "A4")
+  (title_block
+    (company "The A-Team (RC SSL)")
+    (comment 1 "W. Stuckey & R. Osawa")
+  )
   (bus_alias "AIRDRIBBLER" (members "AIRDRIBBLER.PWM1" "AIRDRIBBLER.PWM2"))
   (bus_entry (at 39.37 30.48) (size 2.54 2.54)

Commit message: Update title block
Other:
- title: (none) -> Control
Changed lines of the file:
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@@
   (paper "A4")
   (title_block
+    (title "Control")
+    (date "2024-05-16")
+    (rev "2.0")
     (company "The A-Team (RC SSL)")
     (comment 1 "W. Stuckey & R. Osawa")
