File: robot/control/v2.0.0/control/imu.kicad_sch (KiCad schematic)
At the start: 1 part, among them J5 BM11B-SRSS-TB

Commit message: WIP
Parts:
- added C2 (x2): 0.1uF 63V, Capacitor_SMD:C_0402_1005Metric, symbol Device:C_Small
- added R12 (x2): 100, Resistor_SMD:R_0402_1005Metric, symbol Device:R_Small_US
- added R28 (x2): 4.7k, Resistor_SMD:R_0402_1005Metric, symbol Device:R_Small_US
- added U15: BMI323, AT-IMU:BMI323, symbol AT-IMU:BMI323
Connections:
- net +3.3V: now also C2.1, C2.1, R28.1, R28.1, U15.5 (VDDIO), U15.8 (VDD)
- net GND: now also C2.2, C2.2, U15.6 (GNDIO), U15.7 (GND)
- net IMU.INT1: now also R12.2, R28.2
- net IMU.INT2: now also R12.2, R28.2
- net IMU.MISO: now also U15.1 (SDO)
- net IMU.MOSI: now also U15.14 (SDx)
- net IMU.SCK: now also U15.13 (SCx)
- new net: R12.1, U15.4 (INT1)
- new net: R12.1, U15.9 (INT2)
- new net IMU.~{SS}0: U15.12 (CSB)
Other:
- note added: "On-Board IMU"

Commit message: WIP
Parts:
- renumbered U15 to U16
Changed lines of the file:
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@@
         )
         (path "/e63e39d7-6ac0-4ffd-8aa3-1841a4541b55/3922ffa1-d2bd-44ba-a360-5fe34fca99b4"
-          (reference "#PWR0297") (unit 1)
+          (reference "#PWR0300") (unit 1)
         )
       )
@@
         )
         (path "/e63e39d7-6ac0-4ffd-8aa3-1841a4541b55/3922ffa1-d2bd-44ba-a360-5fe34fca99b4"
+          (reference "#PWR0304") (unit 1)
+        )
+      )
+    )
+  )
+  (symbol (lib_id "power:GND") (at 41.91 57.15 0) (unit 1)
+    (in_bom yes) (on_board yes) (dnp no) (fields_autoplaced)
+    (property "Reference" "#PWR075" (at 41.91 63.5 0)
+      (effects (font (size 1.27 1.27)) hide)
+    )
+    (property "Value" "GND" (at 41.91 62.23 0)
+      (effects (font (size 1.27 1.27)))
+    )
+    (property "Footprint" "" (at 41.91 57.15 0)
+      (effects (font (size 1.27 1.27)) hide)
+    )
+    (property "Datasheet" "" (at 41.91 57.15 0)
+      (effects (font (size 1.27 1.27)) hide)
+    )
+    (pin "1")
+    (instances
+      (project "control"
+        (path "/e63e39d7-6ac0-4ffd-8aa3-1841a4541b55/3a74dea1-1510-40f9-ac26-652aca9a28c3"
+          (reference "#PWR075") (unit 1)
+        )
+        (path "/e63e39d7-6ac0-4ffd-8aa3-1841a4541b55"
+          (reference "#PWR016") (unit 1)
+        )
+        (path "/e63e39d7-6ac0-4ffd-8aa3-1841a4541b55/3922ffa1-d2bd-44ba-a360-5fe34fca99b4"
           (reference "#PWR0301") (unit 1)
-        )
-      )
-    )
-  )
-  (symbol (lib_id "power:GND") (at 41.91 57.15 0) (unit 1)
-    (in_bom yes) (on_board yes) (dnp no) (fields_autoplaced)
-    (property "Reference" "#PWR075" (at 41.91 63.5 0)
-      (effects (font (size 1.27 1.27)) hide)
-    )
-    (property "Value" "GND" (at 41.91 62.23 0)
-      (effects (font (size 1.27 1.27)))
-    )
-    (property "Footprint" "" (at 41.91 57.15 0)
-      (effects (font (size 1.27 1.27)) hide)
-    )
-    (property "Datasheet" "" (at 41.91 57.15 0)
-      (effects (font (size 1.27 1.27)) hide)
-    )
-    (pin "1")
-    (instances
-      (project "control"
-        (path "/e63e39d7-6ac0-4ffd-8aa3-1841a4541b55/3a74dea1-1510-40f9-ac26-652aca9a28c3"
-          (reference "#PWR075") (unit 1)
-        )
-        (path "/e63e39d7-6ac0-4ffd-8aa3-1841a4541b55"
-          (reference "#PWR016") (unit 1)
-        )
-        (path "/e63e39d7-6ac0-4ffd-8aa3-1841a4541b55/3922ffa1-d2bd-44ba-a360-5fe34fca99b4"
-          (reference "#PWR0298") (unit 1)
         )
       )
@@
         )
         (path "/e63e39d7-6ac0-4ffd-8aa3-1841a4541b55/3922ffa1-d2bd-44ba-a360-5fe34fca99b4"
-          (reference "R241") (unit 1)
+          (reference "R243") (unit 1)
         )
       )
@@
         )
         (path "/e63e39d7-6ac0-4ffd-8aa3-1841a4541b55/3922ffa1-d2bd-44ba-a360-5fe34fca99b4"
-          (reference "R239") (unit 1)
+          (reference "R241") (unit 1)
         )
       )
@@
         )
         (path "/e63e39d7-6ac0-4ffd-8aa3-1841a4541b55/3922ffa1-d2bd-44ba-a360-5fe34fca99b4"
-          (reference "R242") (unit 1)
+          (reference "R244") (unit 1)
         )
       )
@@
         )
         (path "/e63e39d7-6ac0-4ffd-8aa3-1841a4541b55/3922ffa1-d2bd-44ba-a360-5fe34fca99b4"
-          (reference "R240") (unit 1)
+          (reference "R242") (unit 1)
         )
       )
@@
         )
         (path "/e63e39d7-6ac0-4ffd-8aa3-1841a4541b55/3922ffa1-d2bd-44ba-a360-5fe34fca99b4"
-          (reference "#PWR0302") (unit 1)
+          (reference "#PWR0305") (unit 1)
         )
       )
@@
         )
         (path "/e63e39d7-6ac0-4ffd-8aa3-1841a4541b55/3922ffa1-d2bd-44ba-a360-5fe34fca99b4"
-          (reference "#PWR0299") (unit 1)
+          (reference "#PWR0302") (unit 1)
         )
       )
@@
         )
         (path "/e63e39d7-6ac0-4ffd-8aa3-1841a4541b55/3922ffa1-d2bd-44ba-a360-5fe34fca99b4"
-          (reference "#PWR0300") (unit 1)
+          (reference "#PWR0303") (unit 1)
         )
       )
@@
   (symbol (lib_id "AT-IMU:BMI323") (at 139.7 38.1 0) (unit 1)
     (in_bom yes) (on_board yes) (dnp no)
-    (property "Reference" "U15" (at 139.7 26.67 0)
+    (property "Reference" "U16" (at 139.7 26.67 0)
       (effects (font (size 1.27 1.27)))
     )
@@
       (project "control"
         (path "/e63e39d7-6ac0-4ffd-8aa3-1841a4541b55/3922ffa1-d2bd-44ba-a360-5fe34fca99b4"
-          (reference "U15") (unit 1)
-        )
-      )
+          (reference "U16") (unit 1)
+        )
+      )

Commit message: Update title block
Other:
- company: (none) -> The A-Team (RC SSL)
Changed lines of the file:
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@@
 (kicad_sch (version 20230121) (generator eeschema)
   (paper "A4")
+  (title_block
+    (company "The A-Team (RC SSL)")
+    (comment 1 "W. Stuckey & R. Osawa")
+  )
   (junction (at 119.38 33.02) (diameter 0) (color 0 0 0 0)
   )

Commit message: Update title block
Other:
- title: (none) -> Control
Changed lines of the file:
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@@
   (paper "A4")
   (title_block
+    (title "Control")
+    (date "2024-05-16")
+    (rev "2.0")
     (company "The A-Team (RC SSL)")
     (comment 1 "W. Stuckey & R. Osawa")
