File: robot/control/v2.0.0/control/indicators.kicad_sch (KiCad schematic)
At the start: 48 parts, among them Q3 BSS138K, Q4 BSS138K, Q5 BSS138K, Q6 BSS138K, Q7 BSS138K, U7 SK9822, U8 SK9822

Commit message: WIP
Parts:
- renumbered R37 to R39, R39 to R41, R40 to R42, R41 to R43, R42 to R44, R43 to R45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

Commit message: WIP
Parts:
- Q4: renamed from Q3; value BSS138K -> SI2310-TP
- renumbered Q4 to Q5, Q5 to Q6, Q6 to Q7, Q7 to Q8, R39 to R41, R41 to R43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
