File: robot/control/v2.0.0/control/optical_flow.kicad_sch (KiCad schematic)
At the start: 1 part, among them J7 BM09B-SRSS-TB

Commit message: Update title block
Other:
- company: (none) -> The A-Team (RC SSL)
Changed lines of the file:
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@@
 (kicad_sch (version 20230121) (generator eeschema)
   (paper "A4")
+  (title_block
+    (company "The A-Team (RC SSL)")
+    (comment 1 "W. Stuckey & R. Osawa")
+  )
   (bus_entry (at 39.37 38.1) (size 2.54 2.54)
     (stroke (width 0) (type default))

Commit message: Update title block
Other:
- title: (none) -> Control
Changed lines of the file:
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@@
   (paper "A4")
   (title_block
+    (title "Control")
+    (date "2024-05-16")
+    (rev "2.0")
     (company "The A-Team (RC SSL)")
     (comment 1 "W. Stuckey & R. Osawa")
