File: robot/kicker/v3.1/kicker/ball_sense.kicad_sch (KiCad schematic)
At the start: 3 parts, among them J4 Conn_01x10

Commit message: Update power entry and regulation
Parts:
- R89, R90: LCSC C60490 -> (none)
Changed lines of the file:
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@@
-      (effects (font (size 1.27 1.27)) hide)
-    )
-    (property "LCSC" "C60490" (at 109.22 41.91 0)
       (effects (font (size 1.27 1.27)) hide)
     )
@@
       (effects (font (size 1.27 1.27)) hide)
     )
-    (property "LCSC" "C60490" (at 100.33 41.91 0)
-      (effects (font (size 1.27 1.27)) hide)
-    )

Commit message: WIP
Parts:
- renumbered R89 to R102, R90 to R103
Changed lines of the file:
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@@
   (symbol (lib_id "Device:R_Small_US") (at 106.68 43.18 0) (unit 1)
     (in_bom yes) (on_board yes) (dnp no) (fields_autoplaced)
-    (property "Reference" "R90" (at 109.22 41.91 0)
+    (property "Reference" "R103" (at 109.22 41.91 0)
       (effects (font (size 1.27 1.27)) (justify left))
     )
@@
       (project "kicker"
         (path "/7c007fad-bfbf-4e78-a837-1f8089552516/7a1ed07f-54d5-4760-ac90-4add0b6ea46f"
-          (reference "R90") (unit 1)
+          (reference "R103") (unit 1)
         )
       )
@@
   (symbol (lib_id "power:GND") (at 118.11 73.66 0) (unit 1)
     (in_bom yes) (on_board yes) (dnp no) (fields_autoplaced)
-    (property "Reference" "#PWR0162" (at 118.11 80.01 0)
+    (property "Reference" "#PWR0174" (at 118.11 80.01 0)
       (effects (font (size 1.27 1.27)) hide)
     )
@@
       (project "kicker"
         (path "/7c007fad-bfbf-4e78-a837-1f8089552516/7a1ed07f-54d5-4760-ac90-4add0b6ea46f"
-          (reference "#PWR0162") (unit 1)
+          (reference "#PWR0174") (unit 1)
         )
       )
@@
   (symbol (lib_id "Device:R_Small_US") (at 97.79 43.18 0) (unit 1)
     (in_bom yes) (on_board yes) (dnp no) (fields_autoplaced)
-    (property "Reference" "R89" (at 100.33 41.91 0)
+    (property "Reference" "R102" (at 100.33 41.91 0)
       (effects (font (size 1.27 1.27)) (justify left))
     )
@@
       (project "kicker"
         (path "/7c007fad-bfbf-4e78-a837-1f8089552516/7a1ed07f-54d5-4760-ac90-4add0b6ea46f"
-          (reference "R89") (unit 1)
+          (reference "R102") (unit 1)
         )
       )
@@
   (symbol (lib_id "power:+3V3") (at 115.57 35.56 0) (unit 1)
     (in_bom yes) (on_board yes) (dnp no) (fields_autoplaced)
-    (property "Reference" "#PWR0161" (at 115.57 39.37 0)
+    (property "Reference" "#PWR0173" (at 115.57 39.37 0)
       (effects (font (size 1.27 1.27)) hide)
     )
@@
       (project "kicker"
         (path "/7c007fad-bfbf-4e78-a837-1f8089552516/7a1ed07f-54d5-4760-ac90-4add0b6ea46f"
-          (reference "#PWR0161") (unit 1)
+          (reference "#PWR0173") (unit 1)
         )
       )
