File: robot/kicker/v3.1/kicker/dribbler.kicad_sch (KiCad schematic)
At the start: 4 parts, among them J12 Conn_01x02, J4 Conn_01x10

Commit message: Update power entry and regulation
Parts:
- J12: LCSC C160403 -> (none)
- R81, R82: LCSC C60490 -> (none)
Changed lines of the file:
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@@
-      (effects (font (size 1.27 1.27)) hide)
-    )
-    (property "LCSC" "C160403" (at 199.39 39.37 0)
       (effects (font (size 1.27 1.27)) hide)
     )
@@
       (effects (font (size 1.27 1.27)) hide)
     )
-    (property "LCSC" "C60490" (at 109.22 40.64 0)
-      (effects (font (size 1.27 1.27)) hide)
-    )
     (pin "1")
     (pin "2")
@@
       (effects (font (size 1.27 1.27)) hide)
     )
-    (property "LCSC" "C60490" (at 119.38 40.64 0)
-      (effects (font (size 1.27 1.27)) hide)
-    )

Commit message: WIP
Parts:
- renumbered R81 to R94, R82 to R95
Changed lines of the file:
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@@
         )
         (path "/7c007fad-bfbf-4e78-a837-1f8089552516/033ff13b-d72f-4800-98f0-39aa58dc7180"
-          (reference "#PWR0144") (unit 1)
+          (reference "#PWR0156") (unit 1)
         )
       )
@@
   (symbol (lib_id "power:+3V3") (at 125.73 34.29 0) (unit 1)
     (in_bom yes) (on_board yes) (dnp no) (fields_autoplaced)
-    (property "Reference" "#PWR0141" (at 125.73 38.1 0)
+    (property "Reference" "#PWR0153" (at 125.73 38.1 0)
       (effects (font (size 1.27 1.27)) hide)
     )
@@
       (project "kicker"
         (path "/7c007fad-bfbf-4e78-a837-1f8089552516/033ff13b-d72f-4800-98f0-39aa58dc7180"
-          (reference "#PWR0141") (unit 1)
+          (reference "#PWR0153") (unit 1)
         )
       )
@@
   (symbol (lib_id "Device:R_Small_US") (at 106.68 41.91 0) (unit 1)
     (in_bom yes) (on_board yes) (dnp no) (fields_autoplaced)
-    (property "Reference" "R81" (at 109.22 40.64 0)
+    (property "Reference" "R94" (at 109.22 40.64 0)
       (effects (font (size 1.27 1.27)) (justify left))
     )
@@
       (project "kicker"
         (path "/7c007fad-bfbf-4e78-a837-1f8089552516/033ff13b-d72f-4800-98f0-39aa58dc7180"
-          (reference "R81") (unit 1)
+          (reference "R94") (unit 1)
         )
       )
@@
   (symbol (lib_id "Device:R_Small_US") (at 116.84 41.91 0) (unit 1)
     (in_bom yes) (on_board yes) (dnp no) (fields_autoplaced)
-    (property "Reference" "R82" (at 119.38 40.64 0)
+    (property "Reference" "R95" (at 119.38 40.64 0)
       (effects (font (size 1.27 1.27)) (justify left))
     )
@@
       (project "kicker"
         (path "/7c007fad-bfbf-4e78-a837-1f8089552516/033ff13b-d72f-4800-98f0-39aa58dc7180"
-          (reference "R82") (unit 1)
+          (reference "R95") (unit 1)
         )
       )
@@
         )
         (path "/7c007fad-bfbf-4e78-a837-1f8089552516/033ff13b-d72f-4800-98f0-39aa58dc7180"
-          (reference "#PWR0142") (unit 1)
+          (reference "#PWR0154") (unit 1)
         )
       )
@@
         )
         (path "/7c007fad-bfbf-4e78-a837-1f8089552516/033ff13b-d72f-4800-98f0-39aa58dc7180"
-          (reference "#PWR0143") (unit 1)
+          (reference "#PWR0155") (unit 1)
         )
       )
