File: robot/power/v1.0/power/voltage_mon.kicad_sch (KiCad schematic)
At the start: 18 parts

Commit message: power board work
Changed lines of the file:
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@@
-		)
-	)
-	(bus
-		(pts
-			(xy 203.2 127) (xy 203.2 129.54)
-		)
-		(stroke
-			(width 0)
-			(type default)
 		)
 	)

Commit message: power schematic work
Changed lines of the file:
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@@
-		)
-	)
-	(label "{VMON}"
-		(at 207.01 110.49 0)
-		(fields_autoplaced yes)
-		(effects
-			(font
-				(size 1.27 1.27)
-			)
-			(justify left bottom)
 		)
 	)
@@
 		)
 	)
-	(global_label "{BATT_BALANCE}"
-		(shape input)
+	(hierarchical_label "{BATT_BALANCE}"
+		(shape bidirectional)
 		(at 39.37 87.63 180)
 		(fields_autoplaced yes)
@@
 			(justify right)
 		)
-		(property "Intersheetrefs" "${INTERSHEET_REFS}"
-			(at 21.2052 87.63 0)
-			(effects
-				(font
-					(size 1.27 1.27)
-				)
-				(justify right)
-				(hide yes)
+	)
+	(hierarchical_label "{VMON}"
+		(shape output)
+		(at 207.01 110.49 0)
+		(fields_autoplaced yes)
+		(effects
+			(font
+				(size 1.27 1.27)
 			)
+			(justify left)
 		)
 	)
