File: robot/control/v3.0/control/control.kicad_pcb (KiCad board)
At the start: 6 copper layers, 148 x 86 mm, 242 parts, among them J1 SD_Card_Device, J10 Conn_01x10_MountingPin, J11 EC3-M, J12 JST-GH-SM05B, J13 Conn_01x04, J14 Conn_01x06, J15 Conn_02x05_Odd_Even, J2 Conn_ARM_JTAG_SWD_10, J3 SM12B-ZESS, J4 BM11B-SRSS-TB, J5 BM10B-SRSS-TB, J6 SM12B-ZESS, J7 SM12B-ZESS, J8 SM12B-ZESS, J9 Conn_01x10_MountingPin, P1 USB_C_Plug_USB2.0, Q1 BSS84, Q2 BSS138K, Q3 SI2310-TP, Q4 BSS138K, SW1 A6SN-1104, SW10 B3F-1000, SW11 B3F-1000, SW12 B3F-1000, SW2 RST, SW3 SW_DIP_x02, SW4 221ADC16, SW5 SW_DIP_x02, SW6 219-8MST, SW7 B3F-1000, SW8 B3F-1000, SW9 B3F-1000, U1 STM32H723ZGTx, U10 SK9822, U11 SK9822, U12 SK9822, U13 SK9822, U14 SK9822, U2 BMI323, U3 TLV70030_SOT353, U4 SK9822, U5 SK9822, U6 SK9822, U7 SK9822, U8 SK9822, U9 SK9822, Y1 Q13FC13500005, Y2 TAXM8M4RDBCCT2T

Commit message: control routing/placement work
Parts:
- C13, R59, R60, R61, R62, R63, R64, R65, R66, R67, R68, R69, R70, R71, R72, R73, R76, R79, R80, R81, R82: moved to B.Cu
- moved R108 112.2 mm to (232.4, 124.3), turned to 180 degrees
- moved R61 111.2 mm to (80.2, 125.0), turned to 180 degrees
- moved R83 110.8 mm to (84.5, 121.3), turned to 90 degrees
- moved R109 109.1 mm to (232.4, 122.3), turned to 180 degrees
- moved R62 109.0 mm to (80.2, 123.7), turned to 180 degrees
- moved R110 106.0 mm to (232.4, 120.3), turned to 180 degrees
- moved R111 103.0 mm to (232.4, 118.3), turned to 180 degrees
- moved R81 95.7 mm to (96.2, 107.8)
- moved R82 89.4 mm to (104.1, 109.3), turned to 90 degrees
- moved R80 88.2 mm to (106.6, 106.2)
- moved R73 87.9 mm to (100.9, 102.7), turned to 90 degrees
- moved R76 86.2 mm to (102.0, 107.3), turned to 90 degrees
- moved R79 83.6 mm to (98.7, 104.7), turned to 90 degrees
- moved R71 82.0 mm to (97.5, 102.5)
- moved R66 81.3 mm to (105.4, 101.0)
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Connections:
- U12 pad 5: Net-(U12-CKO) -> unconnected-(U12-CKO-Pad5)
- U12 pad 6: Net-(U12-SDO) -> unconnected-(U12-SDO-Pad6)
- U13 pad 1: Net-(U12-SDO) -> Net-(U13-SDI)
- U13 pad 2: Net-(U12-CKO) -> Net-(U13-CKI)
- U14 pad 1: Net-(U13-SDO) -> Net-(U14-SDI)
- U14 pad 2: Net-(U13-CKO) -> Net-(U14-CKI)
- U14 pad 5: unconnected-(U14-CKO-Pad5) -> Net-(U13-CKI)
- U14 pad 6: unconnected-(U14-SDO-Pad6) -> Net-(U13-SDI)
- U7 pad 5: Net-(U7-CKO) -> Net-(U14-CKI)
- U7 pad 6: Net-(U7-SDO) -> Net-(U14-SDI)
- U8 pad 1: Net-(U7-SDO) -> Net-(U13-SDO)
- U8 pad 2: Net-(U7-CKO) -> Net-(U13-CKO)
Routing:
- net Net-(U13-SDO): track 9.58 -> 28.9 mm
- net Net-(U13-CKO): track 9.58 -> 27.1 mm
- net Net-(J15-Pin_1): track 0.00 -> 9.16 mm
- net Net-(SW4-8): track 0.00 -> 8.38 mm
- net Net-(R64-Pad1): track 0.00 -> 8.38 mm
- net GND: track 0.04 -> 7.73 mm, vias 45 -> 129
- net Net-(U2-INT1): track 0.00 -> 7.54 mm, vias 0 -> 1
- net +BATT: track 0.00 -> 5.74 mm, vias 0 -> 36
- net Net-(U13-SDI): track 0.00 -> 3.60 mm
- net Net-(U13-CKI): track 0.00 -> 3.60 mm
- net +3V3: track 27.6 -> 30.6 mm, vias 0 -> 36
- net Net-(SW4-4): track 0.00 -> 2.67 mm
- net Net-(SW4-2): track 0.00 -> 2.67 mm
- net Net-(U2-INT2): track 0.00 -> 1.95 mm, vias 0 -> 1
- net /mcu/BOT_ID_DISPLAY.BR: track 0.00 -> 1.80 mm, vias 0 -> 2
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- added copper zone on B.Cu, net +3V3
- added copper zone on In1.Cu, net +3V3
- added copper zone on B.Cu, net +5V
- added copper zone on In4.Cu, net +5V
- added copper zone on F.Cu, net +BATT
- added copper zone on In4.Cu, net +BATT
- added copper zone on F.Cu, net GND
- added copper zone on B.Cu, net Net-(J13-Pin_1)
- added copper zone on F.Cu, net Net-(J13-Pin_1)
- added copper zone on B.Cu, net Net-(J13-Pin_2)
- added copper zone on F.Cu, net Net-(J13-Pin_2)
- added copper zone on F.Cu, net Net-(J3-Pin_1)
- added copper zone on F.Cu, net Net-(J6-Pin_1)
- added copper zone on F.Cu, net Net-(J7-Pin_1)
- added copper zone on F.Cu, net Net-(J8-Pin_1)
Other:
- outline, holes or cut-outs redrawn
- board text added: "A~{U}"
- board text added: "COLOR"
- board text added: "OPTICAL/AUX"
- board text added: "USR1"
- board text added: "USR2"
- board text added: "Y~{B}"
- board text removed: "A"
- board text removed: "B"
- board text removed: "OPTICAL"
- board text removed: "U"
- board text removed: "Y"
