File: robot/power/v1.1/power/output_connectors.kicad_sch (KiCad schematic)
At the start: 12 parts, among them J3 XT60L-F, J4 SM04B-PASS, J6 SM05B-GHS

Commit message: power v1.1 layout work
Parts:
- added J10: SM02B-PASS, AT-Connectors:JST_PA_SM02B-PASS_1x02_P2.00mm_Horizontal, symbol Connector_Generic:Conn_01x02
- added J5: XT30PW-F, Connector_AMASS:AMASS_XT30PW-F_1x02_P2.50mm_Horizontal, symbol Connector_Generic:Conn_01x02
- added J9: SM04B-PASS, AT-Connectors:JST_PA_SM04B-PASS_1x04_P2.00mm_Horizontal, symbol Connector_Generic:Conn_01x04
- J3: value XT60L-F -> XT30PW-F; footprint Connector_AMASS:AMASS_XT60PW-F_1x02_P7.20mm_Horizontal -> Connector_AMASS:AMASS_XT30PW-F_1x02_P2.50mm_Horizontal
Connections:
- net +3.3V: now also J9.2 (Pin_2)
- net +5V: now also J9.1 (Pin_1)
- net +BATT: now also J5.2 (Pin_2)
- net GND: now also J10.1 (Pin_1), J5.1 (Pin_1), J9.3 (Pin_3), J9.4 (Pin_4)
- new net +12V: J10.2 (Pin_2)

Commit message: power v1.1 prod files
Parts:
- J10: LCSC (none) -> C495198
- J4: footprint AT-Connectors:JST_PA_S04B-PASS_1x04_P2.00mm_Horizontal -> AT-Connectors:JST_PA_SM04B-PASS_1x04_P2.00mm_Horizontal
- J6: LCSC (none) -> C189896
- R41, R42, R43: LCSC (none) -> C138034
- R44, R45, R46, R47, R48, R49: LCSC (none) -> C25104
Changed lines of the file:
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@@
+			)
+		)
+		(property "LCSC" "C189896"
+			(at 218.44 77.4699 0)
+			(effects
+				(font
+					(size 1.27 1.27)
+				)
+				(hide yes)
 			)
 		)
@@
 			)
 		)
+		(property "LCSC" "C495198"
+			(at 83.82 118.1101 0)
+			(effects
+				(font
+					(size 1.27 1.27)
+				)
+				(hide yes)
+			)
+		)
 		(pin "2"
 		)
@@
 			)
 		)
+		(property "LCSC" "C138034"
+			(at 176.53 86.3599 0)
+			(effects
+				(font
+					(size 1.27 1.27)
+				)
+				(hide yes)
+			)
+		)
 		(pin "1"
 		)
@@
 			)
 		)
+		(property "LCSC" "C138034"
+			(at 162.56 36.8299 0)
+			(effects
+				(font
+					(size 1.27 1.27)
+				)
+				(hide yes)
+			)
+		)
 		(pin "1"
 		)
@@
 			)
 		)
+		(property "LCSC" "C138034"
+			(at 176.53 36.8299 0)
+			(effects
+				(font
+					(size 1.27 1.27)
+				)
+				(hide yes)
+			)
+		)
 		(pin "1"
 		)
@@
 		(property "Description" "Resistor, small US symbol"
 			(at 187.96 44.45 0)
+			(effects
+				(font
+					(size 1.27 1.27)
+				)
+				(hide yes)
+			)
+		)
+		(property "LCSC" "C25104"
+			(at 187.96 39.116 0)
 			(effects
 				(font
@@
 			)
 		)
-		(property "Footprint" "AT-Connectors:JST_PA_S04B-PASS_1x04_P2.00mm_Horizontal"
+		(property "Footprint" "AT-Connectors:JST_PA_SM04B-PASS_1x04_P2.00mm_Horizontal"
 			(at 81.28 40.64 0)
 			(effects
@@
 			)
 		)
+		(property "LCSC" "C25104"
+			(at 187.96 41.402 0)
+			(effects
+				(font
+					(size 1.27 1.27)
+				)
+				(hide yes)
+			)
+		)
 		(pin "1"
 		)
@@
 			)
 		)
+		(property "LCSC" "C25104"
+			(at 187.96 66.294 0)
+			(effects
+				(font
+					(size 1.27 1.27)
+				)
+				(hide yes)
+			)
+		)
 		(pin "1"
 		)
@@
 			)
 		)
+		(property "LCSC" "C25104"
+			(at 187.96 68.58 0)
+			(effects
+				(font
+					(size 1.27 1.27)
+				)
+				(hide yes)
+			)
+		)
 		(pin "1"
 		)
@@
 			)
 		)
+		(property "LCSC" "C25104"
+			(at 187.96 64.008 0)
+			(effects
+				(font
+					(size 1.27 1.27)
+				)
+				(hide yes)
+			)
+		)
 		(pin "1"
 		)
@@
 			(effects
 				(font
+					(size 1.27 1.27)
+				)
+				(hide yes)
+			)
+		)
+		(property "LCSC" "C25104"
+			(at 187.96 70.866 0)
+			(effects
+				(font
