File: robot/power/v1.1/power/power_protection.kicad_sch (KiCad schematic)
At the start: 34 parts, among them Q3 2N7002, Q4 STL90N10F7, Q5 STL90N10F7, Q6 MMBT5401LT1G, SW2 SM02B-GHS, SW3 CPG151101D91, U4 LM5069, U5 LTC2955-2

Commit message: power v1.1 prod files
Parts:
- C10, C11, C14: LCSC (none) -> C162178
- C12: LCSC (none) -> C415530
- C13: LCSC (none) -> C1848
- D10, D12: LCSC (none) -> C78417
- D11: LCSC (none) -> C241918
- D13: LCSC (none) -> C83528
- Q3: LCSC (none) -> C8545
- Q4, Q5: LCSC (none) -> C457493
- Q6: LCSC (none) -> C231274
- R10: LCSC (none) -> C25896
- R11: LCSC (none) -> C96273
- R12: LCSC (none) -> C26990
- R13: LCSC (none) -> C270576
- R14, R15: LCSC (none) -> C500737
- R16, R21, R9: LCSC (none) -> C11702
- R17, R19, R20: LCSC (none) -> C138034
- R18: LCSC (none) -> C27176
- SW2: LCSC (none) -> C189893
- SW3: LCSC (none) -> C2886902
- U4: LCSC (none) -> C2653582
- U5: LCSC (none) -> C683797
