File: robot/breakbeam/v2.0/breakbeam-receiver/breakbeam-receiver.kicad_sch (KiCad schematic)
At the start: 6 parts, among them J1 Conn_01x03, Q1 OP506B

Commit message: Minor updates
Parts:
- removed J1: Conn_01x03, Connector_JST:JST_SH_SM03B-SRSS-TB_1x03-1MP_P1.00mm_Horizontal, symbol Connector_Generic:Conn_01x03
- added J1: Conn_01x03, Connector_JST:JST_GH_SM03B-GHS-TB_1x03-1MP_P1.25mm_Horizontal, symbol Connector_Generic_MountingPin:Conn_01x03_MountingPin
Connections:
- net +3.3V: now also J1.1 (Pin_1)
- net BALL_RX: now also J1.2 (Pin_2)
- net GND: now also J1.3 (Pin_3)
- no-connect marks 0 -> 1
